File: pcb/hwexla.kicad_pcb (KiCad board)
At the start: 2 copper layers, 60 x 53 mm, 76 parts, among them J1 Conn_01x03, J2 Conn_01x03, J3 DB25_Male, J4 Conn_01x06, J5 Conn_01x04, K1 HFD2/005, Q1 BT148, Q2 2N7002, Q3 2N7002, Q4 2N7002, Q5 2N7002, Q6 2N7002, Q7 BT148, Q8 BT148, SW1 SW_Push, U1 ATtiny1617-M, U2 RR112-1, U3 L78L05_SOT89

Commit message: Use ATmega328 MCU (it fits).
Parts:
- U1: value ATtiny1617-M -> ATmega328P-AU; footprint Package_DFN_QFN:QFN-24-1EP_4x4mm_P0.5mm_EP2.6x2.6mm -> Package_QFP:TQFP-32_7x7mm_P0.8mm
- moved U1 57.1 mm to (31.3, 44.8)
Connections:
- R13 pad 1: /io/L-SLAVE -> (no net)
- R14 pad 1: /io/L-IN+ -> (no net)
- R15 pad 1: /io/L-IN- -> (no net)
- R3 pad 1: VCC -> (no net)
- R3 pad 2: RESET|UPDI -> (no net)
- R4 pad 1: /LED-RED -> (no net)
- R5 pad 1: /LED-YEL -> (no net)
- R6 pad 1: /LED-GR -> (no net)
- U1 pad 1: MAG-SENSE -> (no net)
- U1 pad 10: /io/L-BTN-OUT -> (no net)
- U1 pad 11: /io/L-BTN-IN -> (no net)
- U1 pad 12: /io/L-BTN+OUT -> (no net)
- U1 pad 13: RxD -> (no net)
- U1 pad 14: TxD -> (no net)
- U1 pad 15: /io/L-BTN+IN -> (no net)
- U1 pad 16: /io/L-OUT- -> (no net)
- U1 pad 17: /LED-GR -> (no net)
- U1 pad 18: /LED-YEL -> VCC
- U1 pad 19: /LED-RED -> (no net)
- U1 pad 2: /power/SERVO-POWER-EN -> (no net)
- U1 pad 20: /SERVO-PWM -> (no net)
- U1 pad 21: (no net) -> GND
- U1 pad 22: /BTN -> (no net)
- U1 pad 23: RESET|UPDI -> (no net)
- U1 pad 24: /SERVO-VCC -> (no net)
- U1 pad 25: GND -> (no net)
- U1 pad 5: /io/L-IN+ -> GND
- U1 pad 6: /io/L-IN- -> VCC
- U1 pad 7: /io/L-SLAVE -> (no net)
- U1 pad 8: /io/L-OUT+ -> (no net)
- U1 pad 9: /relay/REL-CONTROL -> (no net)

Commit message: Enhance schematics.
Parts:
- removed the D1 at (38.9, 103.2)
- removed the J2 at (39.4, 93.5)
- added D4: BZX84Cxx, Diode_SMD:D_SOT-23_ANK, F.Cu at (101.5, 58.5)
- added D5: BZX84Cxx, Diode_SMD:D_SOT-23_ANK, F.Cu at (101.5, 63.0)
- added D6: BZX84Cxx, Diode_SMD:D_SOT-23_ANK, F.Cu at (106.0, 58.5)
- added D7: BZX84Cxx, Diode_SMD:D_SOT-23_ANK, F.Cu at (110.4, 58.5)
- D1: renamed from D4; value GREEN -> GR
- D2: renamed from D3; value YELLOW -> YEL
- renumbered C2 to C3, C3 to C4, C4 to C5, C5 to C6, C6 to C7, C7 to C8, C8 to C9, D7 to D10, D8 to D11, D9 to D12, D10 to D13, D11 to D14, D12 to D15, D13 to D16, D14 to D17, D15 to D18, D16 to D19, D2 to D3, D5 to D8, D6 to D9, J3 to J1, J1 to J2, R6 to R3, R5 to R4, R4 to R5, R7 to R6, R3 to R7
Connections:
- D13 pad 1: /SERVO-VCC -> SERVO-VCC
- D16 pad 1: /io/L-BTN-IN -> /L-BTN-IN
- D16 pad 2: /io/L-BTN+IN -> /L-BTN+IN
- F3 pad 1: /SERVO-VCC -> SERVO-VCC
- F7 pad 1: /io/L-BTN+IN -> /L-BTN+IN
- F8 pad 1: /io/L-BTN-IN -> /L-BTN-IN
- J2 pad 1: /SERVO-VCC -> SERVO-VCC
- J5 pad 1: /power/SERVO-POWER-EN -> /SERVO-POWER-EN
- JP1 pad 1: VCC -> (no net)
- JP1 pad 2: Net-(J2-Pad1) -> VCC
- K1 pad 1: /SERVO-VCC -> SERVO-VCC
- Q2 pad 1: /relay/REL-CONTROL -> /REL-CONTROL
- Q3 pad 1: /io/L-BTN+OUT -> /L-BTN+OUT
- Q3 pad 3: /io/L-BTN+IN -> /L-BTN+IN
- Q4 pad 1: /io/L-BTN-OUT -> /L-BTN-OUT
- Q4 pad 3: /io/L-BTN-IN -> /L-BTN-IN
- Q5 pad 1: /io/L-OUT+ -> /L-OUT+
- Q6 pad 1: /io/L-OUT- -> /L-OUT-
- R1 pad 1: /SERVO-PWM -> SERVO-PWM
- R1 pad 2: /SERVO-VCC -> SERVO-VCC
- R11 pad 1: /relay/REL-CONTROL -> /REL-CONTROL
- R13 pad 1: (no net) -> /L-SLAVE
- R14 pad 1: (no net) -> /L-IN+
- R15 pad 1: (no net) -> /L-IN-
- R16 pad 1: /io/L-BTN+OUT -> /L-BTN+OUT
- R17 pad 1: /io/L-BTN-OUT -> /L-BTN-OUT
- R18 pad 1: /io/L-OUT+ -> /L-OUT+
- R19 pad 1: /io/L-OUT- -> /L-OUT-
- R2 pad 2: /SERVO-PWM -> SERVO-PWM
- R3 pad 1: (no net) -> /LED-GR
- R4 pad 1: (no net) -> /LED-YEL
- R5 pad 1: (no net) -> /LED-RED
- R7 pad 1: (no net) -> VCC
- R7 pad 2: (no net) -> RESET
- R9 pad 1: /power/SERVO-POWER-EN -> /SERVO-POWER-EN
- RN1 pad 5: /io/L-BTN+IN -> /L-BTN+IN
- RN1 pad 7: /io/L-BTN-IN -> /L-BTN-IN
- U1 pad 1: (no net) -> /L-BTN-OUT
- U1 pad 10: (no net) -> /LED-YEL
- U1 pad 11: (no net) -> /LED-RED
- U1 pad 12: (no net) -> /SERVO-POWER-EN
- U1 pad 13: (no net) -> SERVO-PWM
- U1 pad 14: (no net) -> /L-IN+
- U1 pad 15: (no net) -> MOSI
- U1 pad 16: (no net) -> MISO
- U1 pad 17: (no net) -> SCK
- U1 pad 2: (no net) -> /REL-CONTROL
- U1 pad 22: (no net) -> MAG-SENSE
- U1 pad 23: (no net) -> SERVO-VCC
- U1 pad 24: (no net) -> /BTN
- U1 pad 25: (no net) -> /L-OUT+
- U1 pad 26: (no net) -> /L-OUT-
- U1 pad 27: (no net) -> /L-BTN+IN
- U1 pad 28: (no net) -> /L-BTN+OUT
- U1 pad 29: (no net) -> RESET
- U1 pad 30: (no net) -> RxD
- U1 pad 31: (no net) -> TxD
- U1 pad 32: (no net) -> /L-BTN-IN
- U1 pad 7: (no net) -> /L-IN-
- U1 pad 8: (no net) -> /L-SLAVE
- U1 pad 9: (no net) -> /LED-GR

Commit message: Use transiles as ESD protection.
Parts:
- removed D7: BZX84Cxx, Diode_SMD:D_SOT-23_ANK
- removed D8, D9: BZX84C5V1, Diode_SMD:D_SOT-23_ANK
- added C2: 100n, Capacitor_SMD:C_0805_2012Metric_Pad1.18x1.45mm_HandSolder, F.Cu at (110.0, 53.5)
- added J3: AVR-ISP-6, Connector_PinSocket_2.54mm:PinSocket_2x03_P2.54mm_Vertical, F.Cu at (105.3, 54.3)
- D4, D5, D6: value BZX84Cxx -> SM05; footprint Diode_SMD:D_SOT-23_ANK -> Package_TO_SOT_SMD:SOT-23
- U3: value L78L05_SOT89 -> KA78M05_TO252; footprint Package_TO_SOT_SMD:SOT-89-3_Handsoldering -> Package_TO_SOT_SMD:TO-252-2
- moved U3 97.5 mm to (125.5, 57.0)
- moved D5 15.8 mm to (114.6, 54.3)
- moved D4 8.41 mm to (109.8, 57.3)
- moved D6 8.33 mm to (114.3, 58.8)
Connections:
- D4 pad 2: GND -> SCK
- D5 pad 1: SCK -> MOSI
- D5 pad 2: GND -> MISO
- D6 pad 1: MOSI -> TxD
- D6 pad 2: GND -> RxD
- JP1 pad 1: (no net) -> Net-(J3-Pad2)
- U1 pad 20: (no net) -> Net-(C2-Pad2)
- U3 pad 1: VCC -> Net-(C6-Pad1)
- U3 pad 3: Net-(C6-Pad1) -> VCC

Commit message: Add pcb dimensions & position servo.
Parts:
- added H1: MountingHole_Pad, MountingHole:MountingHole_2.2mm_M2_Pad_Via, F.Cu at (184.0, 99.5)
- added H2: MountingHole_Pad, MountingHole:MountingHole_2.2mm_M2_Pad_Via, F.Cu at (184.0, 72.0)
- F1: value 50mA -> 200mA
- moved J5 169.8 mm to (194.8, 77.7), turned to 90 degrees
- moved C6 158.0 mm to (195.3, 81.8)
- moved U1 139.8 mm to (164.6, 87.1)
- moved C7 132.8 mm to (181.6, 137.3)
- moved D12 132.8 mm to (163.8, 147.2)
- moved D2 132.8 mm to (180.6, 119.9)
- moved F2 132.8 mm to (174.0, 140.5)
- moved F3 132.8 mm to (174.0, 143.8)
- moved Q1 132.8 mm to (166.1, 141.5)
- moved R1 132.8 mm to (188.9, 125.7)
- moved R10 132.8 mm to (181.8, 134.3)
- moved R2 132.8 mm to (184.1, 125.8)
- moved R3 132.8 mm to (190.1, 119.8)
- moved R4 132.8 mm to (179.4, 122.9)
- moved R5 132.8 mm to (184.1, 122.9)
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Connections:
- J1 pad 1: /IN+ -> /IN-
- J1 pad 12: /RELB- -> /RELB+
- J1 pad 13: /RELB- -> /RELB+
- J1 pad 2: /IN- -> /IN+
- J1 pad 8: /RELB+ -> /RELB-
- J1 pad 9: /RELB+ -> /RELB-
- U1 pad 14: /L-IN+ -> /L-IN-
- U1 pad 7: /L-IN- -> /L-IN+
Routing:
- added copper zone on B.Cu, net GND
- added copper zone on F.Cu, net GND
Other:
- board size 60 x 53 mm -> 53.5 x 53 mm

Commit message: Group footrpints into functional blocks (unwired).
Parts:
- K1: moved to B.Cu
- moved D13 101.7 mm to (214.0, 104.5)
- moved C7 93.3 mm to (232.1, 58.8)
- moved F3 93.3 mm to (224.5, 65.3)
- moved C5 93.3 mm to (209.4, 68.7)
- moved R10 93.3 mm to (232.3, 55.8)
- moved R9 93.3 mm to (219.0, 68.6)
- moved D12 93.3 mm to (214.3, 68.7)
- moved F2 84.5 mm to (199.5, 60.0), turned to 90 degrees
- moved Q1 82.3 mm to (202.0, 67.5), turned to 270 degrees
- moved Q2 79.8 mm to (214.0, 100.0)
- moved R11 79.7 mm to (214.0, 108.5)
- moved D10 73.3 mm to (192.0, 66.5), turned to 270 degrees
- moved F1 67.1 mm to (178.5, 50.0)
- moved D5 59.9 mm to (163.5, 111.0)
- moved D6 59.1 mm to (169.0, 111.0)
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
Commit message: Add protective resistors to L-BTN, add C to overvolt. prot.
Parts:
- added C10: 100n, Capacitor_SMD:C_0805_2012Metric_Pad1.18x1.45mm_HandSolder, F.Cu at (196.0, 63.5)
- added C11: 100n, Capacitor_SMD:C_0805_2012Metric_Pad1.18x1.45mm_HandSolder, F.Cu at (149.5, 69.5)
- added C12: 100n, Capacitor_SMD:C_0805_2012Metric_Pad1.18x1.45mm_HandSolder, F.Cu at (149.5, 57.5)
- added R22: 2k2, Resistor_SMD:R_0805_2012Metric_Pad1.20x1.40mm_HandSolder, F.Cu at (132.0, 76.5)
- added R23: 2k2, Resistor_SMD:R_0805_2012Metric_Pad1.20x1.40mm_HandSolder, F.Cu at (136.8, 76.5)
- moved D11 32.6 mm to (195.5, 135.5)
- moved U2 32.4 mm to (184.0, 105.0), turned to 270 degrees
Connections:
- D16 pad 1: /L-BTN-IN -> Net-(D16-Pad1)
- D16 pad 2: /L-BTN+IN -> Net-(D16-Pad2)
- F7 pad 1: /L-BTN+IN -> Net-(D16-Pad2)
- F8 pad 1: /L-BTN-IN -> Net-(D16-Pad1)
- Q3 pad 3: /L-BTN+IN -> Net-(D16-Pad2)
- Q4 pad 3: /L-BTN-IN -> Net-(D16-Pad1)
- RN1 pad 5: /L-BTN+IN -> Net-(D16-Pad2)
- RN1 pad 7: /L-BTN-IN -> Net-(D16-Pad1)
Routing:
- added copper zone on In1.Cu, net GND
Other:
- copper layers 2 -> 4

Commit message: Wire part of PCB.
Parts:
- removed D12: 1N4148, Diode_SMD:D_0805_2012Metric_Pad1.15x1.40mm_HandSolder
- removed R14, R15, R22, R23: 2k2, Resistor_SMD:R_0805_2012Metric_Pad1.20x1.40mm_HandSolder
- removed R16, R17, R18, R19: 10k, Resistor_SMD:R_0805_2012Metric_Pad1.20x1.40mm_HandSolder
- added D7: 1N4007, Diode_SMD:D_SOD-123, F.Cu at (177.8, 53.6)
- added RN2: 2k2, Resistor_SMD:R_Array_Concave_4x0603, F.Cu at (169.9, 78.7)
- added RN3: 10k, Resistor_SMD:R_Array_Concave_4x0603, F.Cu at (168.4, 73.7)
- C11, C12, C8, C9, D14, D15, D16, D17, D18, D19, F2, Q7, Q8, R20, R21: moved to B.Cu
- moved RN1 82.4 mm to (191.0, 54.4), turned to 90 degrees
- moved F6 76.6 mm to (196.3, 63.8), turned to 90 degrees
- moved F10 76.3 mm to (185.4, 63.8), turned to 90 degrees
- moved F9 75.9 mm to (188.2, 63.8), turned to 90 degrees
- moved D17 74.1 mm to (185.7, 50.5), turned to 90 degrees
- moved F5 72.4 mm to (193.7, 63.8), turned to 90 degrees
- moved F4 68.3 mm to (191.0, 63.8), turned to 90 degrees
- moved D15 67.6 mm to (196.1, 50.5), turned to 90 degrees
- moved F8 66.4 mm to (179.8, 63.8), turned to 90 degrees
- moved F7 66.3 mm to (182.6, 63.8), turned to 90 degrees
- moved D16 63.9 mm to (184.7, 52.8), turned to 90 degrees
- moved D14 60.4 mm to (190.8, 50.5), turned to 90 degrees
- moved K1 56.1 mm to (159.5, 74.0), turned to 90 degrees
- moved Q6 55.0 mm to (172.7, 71.6), turned to 90 degrees
- moved Q5 54.1 mm to (176.5, 71.6), turned to 90 degrees
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Connections:
- RN1 pad 2: VCC -> Net-(D15-Pad1)
- RN1 pad 3: Net-(D15-Pad1) -> Net-(D16-Pad2)
- RN1 pad 4: VCC -> Net-(D16-Pad1)
- RN1 pad 5: Net-(D16-Pad2) -> VCC
- RN1 pad 7: Net-(D16-Pad1) -> VCC
Routing:
- net Net-(D15-Pad2): track 0.00 -> 35.2 mm, vias 0 -> 2
- net Net-(D15-Pad1): track 0.00 -> 31.6 mm, vias 0 -> 2
- net /RELB-: track 0.00 -> 31.5 mm
- net Net-(D14-Pad1): track 0.00 -> 25.9 mm, vias 0 -> 2
- net /RELA-: track 0.00 -> 25.6 mm
- net Net-(D16-Pad2): track 0.00 -> 25.4 mm, vias 0 -> 2
- net /RELA+: track 0.00 -> 22.7 mm
- net +12V: track 0.00 -> 21.1 mm
- net /RELB+: track 0.00 -> 20.8 mm
- net Net-(D16-Pad1): track 0.00 -> 20.2 mm, vias 0 -> 2
- net /RELB0: track 0.00 -> 20.2 mm, vias 0 -> 4
- net Net-(D17-Pad1): track 0.00 -> 18.5 mm, vias 0 -> 2
- net /RELA0: track 0.00 -> 14.4 mm
- net Net-(D17-Pad2): track 0.00 -> 14.3 mm
- net /power/STEPIN: track 0.00 -> 11.2 mm
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Other:
- net class Trakce added: clearance 0.2, trace_width 2.5, via_dia 0.8, via_drill 0.4
- rule via_min_size: 0.4 -> 0.3

Commit message: Place IO protection.
Parts:
- moved Q8 73.6 mm to (197.4, 84.8)
- moved D19 69.1 mm to (198.4, 90.7)
- moved Q7 68.9 mm to (197.4, 72.9)
- moved R21 62.5 mm to (195.3, 90.7)
- moved D18 62.4 mm to (198.4, 78.7)
- moved C12 61.7 mm to (201.4, 90.7)
- moved C9 57.5 mm to (193.0, 90.7), turned to 90 degrees
- moved U3 56.4 mm to (216.4, 72.6), turned to 180 degrees
- moved R20 54.4 mm to (195.3, 78.7)
- moved C11 53.5 mm to (201.4, 78.7), turned to 90 degrees
- moved C8 48.7 mm to (193.0, 78.7), turned to 90 degrees
- moved J5 22.3 mm to (202.2, 98.8), turned to 270 degrees
- moved R10 16.6 mm to (201.4, 78.2), turned to 270 degrees
- moved D11 16.2 mm to (196.1, 78.2), turned to 180 degrees
- moved D17 15.8 mm to (187.5, 66.3), turned to 270 degrees
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Connections:
- F5 pad 1: Net-(D15-Pad2) -> Net-(D15-Pad1)
- F6 pad 1: Net-(D15-Pad1) -> Net-(D15-Pad2)
- RN1 pad 1: Net-(D15-Pad2) -> Net-(D15-Pad1)
- RN1 pad 2: Net-(D15-Pad1) -> Net-(D15-Pad2)
- RN2 pad 1: Net-(D15-Pad1) -> Net-(D15-Pad2)
- RN2 pad 2: Net-(D15-Pad2) -> Net-(D15-Pad1)
Routing:
- net Net-(C12-Pad2): track 0.00 -> 40.3 mm, vias 0 -> 4
- net Net-(C11-Pad1): track 0.00 -> 32.2 mm
- net /power/STEPIN: track 11.2 -> 32.8 mm
- net Net-(D15-Pad1): track 31.6 -> 40.5 mm, vias 2 -> 5
- net Net-(D16-Pad1): track 20.2 -> 26.0 mm, vias 2 -> 4
- net Net-(C9-Pad1): track 0.00 -> 4.37 mm
- net Net-(C8-Pad1): track 0.00 -> 4.37 mm
- net Net-(D17-Pad1): track 18.5 -> 22.3 mm, vias 2 -> 3
- net Net-(D16-Pad2): track 25.4 -> 28.8 mm, vias 2 -> 3
- net Net-(D17-Pad2): track 14.3 -> 17.7 mm, vias 0 -> 2
- net Net-(D14-Pad1): track 25.9 -> 28.7 mm, vias 2 -> 4
- net Net-(D15-Pad2): track 35.2 -> 36.0 mm, vias 2 -> 4
