File: pcb/hwexla.kicad_pcb (KiCad board)
At the start: 4 copper layers, 53.5 x 53 mm, 78 parts, among them J1 DB25_Male, J2 Conn_01x03, J3 AVR-ISP-6, J4 Conn_01x06, J5 Conn_01x04, K1 HFD2/005, Q1 BT148, Q2 2N7002, Q3 2N7002, Q4 2N7002, Q5 2N7002, Q6 2N7002, Q7 BT148, Q8 BT148, SW1 SW_Push, U1 ATmega8A-AU, U2 RR112-1, U3 KA78M05_TO252

Commit message: Add alternate MCUs, add testpoints.
Parts:
- added TP1: TestPoint, TestPoint:TestPoint_Pad_D1.5mm, B.Cu at (168.4, 90.4)
- C6: value 22u -> 22u/25V
- C7: value 22u -> 47u
Connections:
- U1 pad 19: (no net) -> Net-(TP1-Pad1)
Routing:
- net Net-(TP1-Pad1): track 0.00 -> 4.11 mm, vias 0 -> 1

Commit message: Add GND testpoint.
Parts:
- added TP2: TestPoint, TestPoint:TestPoint_Loop_D3.50mm_Drill1.4mm_Beaded, F.Cu at (189.6, 97.3)
Changed lines of the file:
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@@
     (tracks 794)
     (zones 0)
-    (modules 79)
+    (modules 80)
     (nets 67)
   )
@@
     (add_net /RELB0)
   )
+  (module TestPoint:TestPoint_Loop_D3.50mm_Drill1.4mm_Beaded (layer F.Cu)
+    (at 189.611 97.282)
+    (descr "wire loop with bead as test point, loop diameter 3.5mm, hole diameter 1.4mm")
+    (tags "test point wire loop bead")
+    (fp_text reference TP2 (at -2.667 0 90) (layer F.SilkS)
+      (effects (font (size 1 1) (thickness 0.15)))
+    )
+    (fp_text value TestPoint (at 0 -2.8) (layer F.Fab)
+      (effects (font (size 1 1) (thickness 0.15)))
+    )
+    (fp_text user %R (at 0.7 2.5) (layer F.Fab)
+      (effects (font (size 1 1) (thickness 0.15)))
+    )
+    (fp_line (start -1.6 -0.3) (end -1.6 0.3) (layer F.Fab) (width 0.12))
+    (fp_line (start -1.6 0.3) (end 1.6 0.3) (layer F.Fab) (width 0.12))
+    (fp_line (start 1.6 0.3) (end 1.6 -0.3) (layer F.Fab) (width 0.12))
+    (fp_line (start 1.6 -0.3) (end -1.6 -0.3) (layer F.Fab) (width 0.12))
+    (fp_circle (center 0 0) (end 2.1 0) (layer F.CrtYd) (width 0.05))
+    (fp_circle (center 0 0) (end 1.8 0) (layer F.SilkS) (width 0.12))
+    (fp_circle (center 0 0) (end 1.5 0) (layer F.Fab) (width 0.12))
+    (pad 1 thru_hole circle (at 0 0) (size 2.8 2.8) (drill 1.4) (layers *.Cu *.Mask)
+      (net 2 GND))
+    (model ${KISYS3DMOD}/TestPoint.3dshapes/TestPoint_Loop_D3.50mm_Drill1.4mm_Beaded.wrl
+      (at (xyz 0 0 0))
+      (scale (xyz 1 1 1))
+      (rotate (xyz 0 0 0))
+    )
+  )
   (module TestPoint:TestPoint_Pad_D1.5mm (layer B.Cu)
     (at 168.402 90.424)
@@
     (tags "test point SMD pad")
     (attr virtual)
-    (fp_text reference TP1 (at 0.381 2.54 90) (layer B.SilkS)
+    (fp_text reference TP1 (at 3.683 0 180) (layer B.SilkS)
       (effects (font (size 1 1) (thickness 0.15)) (justify mirror))
     )
@@
     (attr smd)
     (fp_text reference D2 (at -2.402 -0.015 180) (layer F.SilkS)
-      (effects (font (size 1 1) (thickness 0.15)))
+      (effects (font (size 0.8 0.8) (thickness 0.15)))
     )
     (fp_text value YEL (at 0 1.65 90) (layer F.Fab)
@@
     (tags "capacitor handsolder")
     (attr smd)
-    (fp_text reference C4 (at 3.206 0.015 90) (layer F.SilkS)
+    (fp_text reference C4 (at 2.952 0.015 90) (layer F.SilkS)
       (effects (font (size 1 1) (thickness 0.15)))
     )
@@
     (tags "capacitor handsolder")
     (attr smd)
-    (fp_text reference C3 (at 3.017 0.112 90) (layer F.SilkS)
+    (fp_text reference C3 (at -2.825 -0.015 90) (layer F.SilkS)
       (effects (font (size 1 1) (thickness 0.15)))
     )

Commit message: Add openhardware logo.
Parts:
- added REF**: OSHW-Symbol_8.9x8mm_SilkScreen, Symbol:OSHW-Symbol_8.9x8mm_SilkScreen, B.Cu at (170.4, 73.0)
Routing:
- net /power/STEPIN: track 60.6 -> 61.6 mm
Other:
- board text added: "open hardware"

Commit message: Add MOSFET gate protection resistors.
Parts:
- removed the REF** at (170.4, 73.0)
- added REF**: OSHW-Symbol_6.7x6mm_SilkScreen, Symbol:OSHW-Symbol_6.7x6mm_SilkScreen, B.Cu at (174.6, 66.2)
- added RN4: 250R, Resistor_SMD:R_Array_Concave_4x0603, B.Cu at (174.2, 76.1)
Connections:
- Q3 pad 1: /L-BTN+OUT -> Net-(Q3-Pad1)
- Q4 pad 1: /L-BTN-OUT -> Net-(Q4-Pad1)
- Q5 pad 1: /L-OUT+ -> Net-(Q5-Pad1)
- Q6 pad 1: /L-OUT- -> Net-(Q6-Pad1)
- RN3 pad 5: /L-OUT+ -> Net-(Q5-Pad1)
- RN3 pad 6: /L-OUT- -> Net-(Q6-Pad1)
- RN3 pad 7: /L-BTN-OUT -> Net-(Q4-Pad1)
- RN3 pad 8: /L-BTN+OUT -> Net-(Q3-Pad1)
Routing:
- net /L-BTN-OUT: track 35.6 -> 17.0 mm
- net Net-(Q4-Pad1): track 0.00 -> 16.9 mm, vias 0 -> 1
- net /L-BTN+OUT: track 33.7 -> 18.6 mm
- net Net-(Q3-Pad1): track 0.00 -> 13.3 mm, vias 0 -> 1
- net /L-OUT-: track 34.1 -> 22.9 mm
- net Net-(Q6-Pad1): track 0.00 -> 9.50 mm, vias 0 -> 1
- net /L-OUT+: track 30.0 -> 21.8 mm
- net Net-(Q5-Pad1): track 0.00 -> 6.57 mm, vias 0 -> 1
- net VCC: vias 20 -> 19

Commit message: Debug: use pinsocket instead of pinheader.
Parts:
- removed REF**: OSHW-Symbol_6.7x6mm_SilkScreen, Symbol:OSHW-Symbol_6.7x6mm_SilkScreen
- J4: footprint Connector_PinHeader_2.54mm:PinHeader_1x06_P2.54mm_Vertical -> Connector_PinSocket_2.54mm:PinSocket_1x06_P2.54mm_Vertical

Commit message: Fix too long net.
Routing:
- net SCK: track 19.6 -> 19.1 mm
- net MOSI: track 20.8 -> 20.3 mm
Changed lines of the file:
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@@
   )
   (setup
-    (last_trace_width 0.25)
+    (last_trace_width 0.4)
     (user_trace_width 0.3)
     (user_trace_width 0.4)
@@
     (add_net "Net-(D13-Pad2)")
     (add_net "Net-(D14-Pad1)")
-    (add_net "Net-(D14-Pad2)")
     (add_net "Net-(D15-Pad1)")
     (add_net "Net-(D15-Pad2)")
@@
     (add_net "Net-(D2-Pad2)")
     (add_net "Net-(D3-Pad2)")
-    (add_net "Net-(D4-Pad3)")
-    (add_net "Net-(D5-Pad1)")
-    (add_net "Net-(D5-Pad3)")
-    (add_net "Net-(D5-Pad5)")
     (add_net "Net-(F1-Pad2)")
-    (add_net "Net-(J1-Pad18)")
     (add_net "Net-(J2-Pad3)")
     (add_net "Net-(J3-Pad2)")
-    (add_net "Net-(J4-Pad1)")
     (add_net "Net-(J4-Pad4)")
-    (add_net "Net-(J4-Pad5)")
     (add_net "Net-(Q3-Pad1)")
     (add_net "Net-(Q4-Pad1)")
@@
   (segment (start 172.286 92.558) (end 172.286 94.48699) (width 0.4) (layer F.Cu) (net 35) (status 10))
   (segment (start 172.286 94.48699) (end 171.80799 94.965) (width 0.4) (layer F.Cu) (net 35))
-  (segment (start 162.418 100.71) (end 162.956 100.172) (width 0.4) (layer F.Cu) (net 35) (status 30))
-  (segment (start 162.418 103.444) (end 162.418 100.71) (width 0.4) (layer F.Cu) (net 35) (status 20))
+  (segment (start 162.418 100.71) (end 162.418 102.936) (width 0.4) (layer F.Cu) (net 35))
+  (segment (start 162.956 100.172) (end 162.418 100.71) (width 0.4) (layer F.Cu) (net 35))
   (segment (start 164.245999 98.921999) (end 166.212495 98.921999) (width 0.4) (layer B.Cu) (net 36))
   (via (at 169.940996 92.171) (size 0.6) (drill 0.3) (layers F.Cu B.Cu) (net 36))
@@
   (segment (start 164.226 100.823) (end 164.226 98.902) (width 0.4) (layer F.Cu) (net 36))
   (segment (start 163.068 101.981) (end 164.226 100.823) (width 0.4) (layer F.Cu) (net 36))
-  (segment (start 163.068 103.444) (end 163.068 101.981) (width 0.4) (layer F.Cu) (net 36))
+  (segment (start 163.068 101.981) (end 163.068 102.936) (width 0.4) (layer F.Cu) (net 36))
   (segment (start 165.938 100.614) (end 165.496 100.172) (width 0.4) (layer F.Cu) (net 37) (status 30))
   (segment (start 165.496 101.158) (end 165.496 100.172) (width 0.4) (layer F.Cu) (net 37) (status 20))

Commit message: Add OSHW logo.
Parts:
- added REF**: OSHW-Symbol_6.7x6mm_SilkScreen, Symbol:OSHW-Symbol_6.7x6mm_SilkScreen, B.Cu at (174.6, 66.3)

Commit message: Migrate to KiCad 6.
Other:
- net class Default removed
- net class Trakce removed
