File: pcb/hwexla.kicad_pcb (KiCad board)
At the start: 4 copper layers, 53.5 x 53 mm, 82 parts, among them J1 DB25_Male, J2 Conn_01x03, J3 AVR-ISP-6, J4 Conn_01x06, J5 Conn_01x04, K1 HFD2/005, Q1 BT148, Q2 2N7002, Q3 2N7002, Q4 2N7002, Q5 2N7002, Q6 2N7002, Q7 BT148, Q8 BT148, SW1 SW_Push, U1 ATmega8A-AU, U2 RR112-1, U3 KA78M05_TO252

Commit message: Use net between IO & MCU to make schematics more clear.
Parts:
- removed REF**: OSHW-Logo_7.5x8mm_SilkScreen, Symbol:OSHW-Logo_7.5x8mm_SilkScreen

Commit message: Allow using of SOT353 TVS.
Parts:
- RN4: value 250R -> 470R
Connections:
- D4 pad 3: unconnected-(D4-Pad3) -> MOSI
Routing:
- net MOSI: track 20.7 -> 22.8 mm
- net GND: vias 98 -> 96
Changed lines of the file:
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@@
   (net 68 "Net-(Q5-Pad1)")
   (net 69 "Net-(Q6-Pad1)")
-  (net 70 "unconnected-(D4-Pad3)")
-  (net 71 "unconnected-(D5-Pad1)")
-  (net 72 "unconnected-(D5-Pad3)")
-  (net 73 "unconnected-(D5-Pad5)")
-  (net 74 "unconnected-(D14-Pad2)")
-  (net 75 "unconnected-(J1-Pad18)")
-  (net 76 "unconnected-(J4-Pad1)")
-  (net 77 "unconnected-(J4-Pad5)")
+  (net 70 "unconnected-(D5-Pad1)")
+  (net 71 "unconnected-(D5-Pad3)")
+  (net 72 "unconnected-(D5-Pad5)")
+  (net 73 "unconnected-(D14-Pad2)")
+  (net 74 "unconnected-(J1-Pad18)")
+  (net 75 "unconnected-(J4-Pad1)")
+  (net 76 "unconnected-(J4-Pad5)")
   (footprint "Resistor_SMD:R_0805_2012Metric_Pad1.20x1.40mm_HandSolder" (layer "F.Cu")
     (at 201.93 99.822)
@@
     (fp_line (start 0.635 -1.27) (end 1.27 -0.635) (layer "F.Fab") (width 0.1))
     (pad "1" thru_hole rect locked (at 0 0) (size 1.7 1.7) (drill 1) (layers *.Cu *.Mask)
-      (net 76 "unconnected-(J4-Pad1)") (pinfunction "Pin_1") (pintype "passive+no_connect"))
+      (net 75 "unconnected-(J4-Pad1)") (pinfunction "Pin_1") (pintype "passive+no_connect"))
     (pad "2" thru_hole oval locked (at 0 2.54) (size 1.7 1.7) (drill 1) (layers *.Cu *.Mask)
       (net 8 "TxD") (pinfunction "Pin_2") (pintype "passive"))
@@
       (net 28 "Net-(J4-Pad4)") (pinfunction "Pin_4") (pintype "passive"))
     (pad "5" thru_hole oval locked (at 0 10.16) (size 1.7 1.7) (drill 1) (layers *.Cu *.Mask)
-      (net 77 "unconnected-(J4-Pad5)") (pinfunction "Pin_5") (pintype "passive+no_connect"))
+      (net 76 "unconnected-(J4-Pad5)") (pinfunction "Pin_5") (pintype "passive+no_connect"))
     (pad "6" thru_hole oval locked (at 0 12.7) (size 1.7 1.7) (drill 1) (layers *.Cu *.Mask)
       (net 2 "GND") (pinfunction "Pin_6") (pintype "passive"))
@@
       (net 13 "+12V") (pinfunction "P17") (pintype "passive"))
     (pad "18" smd rect locked (at -4.155 0 180) (size 1.846667 3.48) (layers "B.Cu" "B.Paste" "B.Mask")
-      (net 75 "unconnected-(J1-Pad18)") (pinfunction "P18") (pintype "passive+no_connect"))
+      (net 74 "unconnected-(J1-Pad18)") (pinfunction "P18") (pintype "passive+no_connect"))
     (pad "19" smd rect locked (at -1.385 0 180) (size 1.846667 3.48) (layers "B.Cu" "B.Paste" "B.Mask")
       (net 12 "Net-(F1-Pad2)") (pinfunction "P19") (pintype "passive"))
@@
       (net 2 "GND") (pinfunction "A") (pintype "passive"))
     (pad "3" smd rect locked (at -0.95 0.65 90) (size 0.65 0.4) (layers "F.Cu" "F.Paste" "F.Mask")
-      (net 70 "unconnected-(D4-Pad3)") (pinfunction "K") (pintype "passive+no_connect"))
+      (net 36 "MOSI") (pinfunction "K") (pintype "passive"))
     (pad "4" smd rect locked (at 0.95 0.65 90) (size 0.65 0.4) (layers "F.Cu" "F.Paste" "F.Mask")
       (net 37 "MISO") (pinfunction "K") (pintype "passive"))
@@
     (fp_line (start -0.175 -1.1) (end -0.675 -0.6) (layer "F.Fab") (width 0.1))
     (pad "1" smd rect locked (at -0.95 -0.65 270) (size 0.65 0.4) (layers "F.Cu" "F.Paste" "F.Mask")
-      (net 71 "unconnected-(D5-Pad1)") (pinfunction "K") (pintype "passive+no_connect"))
+      (net 70 "unconnected-(D5-Pad1)") (pinfunction "K") (pintype "passive+no_connect"))
     (pad "2" smd rect locked (at -0.95 0 270) (size 0.65 0.4) (layers "F.Cu" "F.Paste" "F.Mask")
       (net 2 "GND") (pinfunction "A") (pintype "passive"))
     (pad "3" smd rect locked (at -0.95 0.65 270) (size 0.65 0.4) (layers "F.Cu" "F.Paste" "F.Mask")
-      (net 72 "unconnected-(D5-Pad3)") (pinfunction "K") (pintype "passive+no_connect"))
+      (net 71 "unconnected-(D5-Pad3)") (pinfunction "K") (pintype "passive+no_connect"))
     (pad "4" smd rect locked (at 0.95 0.65 270) (size 0.65 0.4) (layers "F.Cu" "F.Paste" "F.Mask")
       (net 8 "TxD") (pinfunction "K") (pintype "passive"))
     (pad "5" smd rect locked (at 0.95 0 270) (size 0.65 0.4) (layers "F.Cu" "F.Paste" "F.Mask")
-      (net 73 "unconnected-(D5-Pad5)") (pinfunction "K") (pintype "passive+no_connect"))
+      (net 72 "unconnected-(D5-Pad5)") (pinfunction "K") (pintype "passive+no_connect"))
     (pad "6" smd rect locked (at 0.95 -0.65 270) (size 0.65 0.4) (layers "F.Cu" "F.Paste" "F.Mask")
       (net 9 "RxD") (pinfunction "K") (pintype "passive"))
@@
       (net 11 "Net-(D14-Pad1)") (pintype "passive"))
     (pad "2" smd roundrect locked (at -0.9375 -0.95 270) (size 1.475 0.6) (layers "B.Cu" "B.Paste" "B.Mask") (roundrect_rratio 0.25)
-      (net 74 "unconnected-(D14-Pad2)") (pintype "passive+no_connect"))
+      (net 73 "unconnected-(D14-Pad2)") (pintype "passive+no_connect"))
     (pad "3" smd roundrect locked (at 0.9375 0 270) (size 1.475 0.6) (layers "B.Cu" "B.Paste" "B.Mask") (roundrect_rratio 0.25)
       (net 59 "Net-(D16-Pad2)") (pintype "passive"))
@@
       (effects (font (size 1 1) (thickness 0.15)) (justify mirror))
     )
-    (fp_text value "250R" (at 0 -2.6 -90) (layer "B.Fab")
+    (fp_text value "470R" (at 0 -2.6 -90) (layer "B.Fab")
       (effects (font (size 1 1) (thickness 0.15)) (justify mirror))
     )
@@
   (via (at 193.675 82.423) (size 0.8) (drill 0.4) (layers "F.Cu" "B.Cu") (net 2))
   (via (at 159.004 80.645) (size 0.6) (drill 0.3) (layers "F.Cu" "B.Cu") (free) (net 2))
-  (via (at 163.957 104.267) (size 0.6) (drill 0.3) (layers "F.Cu" "B.Cu") (net 2))
   (via (at 192.151 76.073) (size 0.8) (drill 0.4) (layers "F.Cu" "B.Cu") (net 2))
   (via (at 154.686 85.217) (size 0.6) (drill 0.3) (layers "F.Cu" "B.Cu") (net 2))
@@
   (via (at 170.815 90.17) (size 0.6) (drill 0.3) (layers "F.Cu" "B.Cu") (net 2))
   (via (at 181.991 103.759) (size 0.6) (drill 0.3) (layers "F.Cu" "B.Cu") (net 2))
-  (via (at 163.068 104.267) (size 0.6) (drill 0.3) (layers "F.Cu" "B.Cu") (net 2))
   (via (at 192.151 70.104) (size 0.8) (drill 0.4) (layers "F.Cu" "B.Cu") (net 2))
   (via (at 191.135 68.072) (size 0.8) (drill 0.4) (layers "F.Cu" "B.Cu") (net 2))
@@
   (segment (start 171.80799 96.920008) (end 171.80799 94.965) (width 0.4) (layer "B.Cu") (net 35))
   (segment (start 162.956 100.172) (end 164.226 101.442) (width 0.4) (layer "B.Cu") (net 35))
+  (segment (start 163.068 104.042) (end 163.718 104.692) (width 0.4) (layer "F.Cu") (net 36))
+  (segment (start 163.068 103.317) (end 163.068 104.042) (width 0.4) (layer "F.Cu") (net 36))
   (segment (start 169.940996 93.912996) (end 169.940996 92.171) (width 0.4) (layer "F.Cu") (net 36))
   (segment (start 163.068 101.981) (end 163.068 103.317) (width 0.4) (layer "F.Cu") (net 36))
+  (segment (start 163.718 104.692) (end 163.718 105.217) (width 0.4) (layer "F.Cu") (net 36))
   (segment (start 164.226 100.823) (end 163.068 101.981) (width 0.4) (layer "F.Cu") (net 36))
   (segment (start 164.226 98.902) (end 164.226 100.823) (width 0.4) (layer "F.Cu") (net 36))

Commit message: v1.1 initial change
Other:
- board text added: "hWexla v1.1 KMŽ Brno I JH 2022"
- board text removed: "hWexla v1.0 KMŽ Brno I JH 2022"
Changed lines of the file:
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@@
   (gr_line (start 152.634 60.556) (end 152.634 105.056) (layer "Edge.Cuts") (width 0.05))
   (gr_line (start 154.634 107.056) (end 204.134 107.056) (layer "Edge.Cuts") (width 0.05))
-  (gr_text "hWexla v1.0\nKMŽ Brno I\nJH 2022" (at 164.211 86.106) (layer "B.SilkS")
+  (gr_text "hWexla v1.1\nKMŽ Brno I\nJH 2022" (at 164.211 86.106) (layer "B.SilkS")
     (effects (font (size 1.3 1.3) (thickness 0.2)) (justify mirror))
   )

Commit message: Add missing OSHW logo.
Parts:
- added REF**: OSHW-Logo_7.5x8mm_SilkScreen, Symbol:OSHW-Logo_7.5x8mm_SilkScreen, B.Cu at (172.5, 68.6)
Connections:
- C11 pad 1: Net-(D16-Pad2) -> Net-(C11-Pad1)
- D14 pad 3: Net-(D16-Pad2) -> Net-(C11-Pad1)
- D15 pad 3: Net-(D16-Pad2) -> Net-(C11-Pad1)
- D16 pad 3: Net-(D16-Pad2) -> Net-(C11-Pad1)
- D18 pad 1: Net-(D16-Pad2) -> Net-(C11-Pad1)
- Q7 pad 1: Net-(D16-Pad2) -> Net-(C11-Pad1)
Routing:
- net Net-(D16-Pad2): track 67.9 -> 0.00 mm, vias 4 -> 0
- net Net-(C11-Pad1): track 0.00 -> 67.9 mm, vias 0 -> 4

Commit message: Fix bad BT148 pinout & fix connected wires.
Connections:
- Q1 pad 1: /power/STEPIN -> GND
- Q1 pad 2: Net-(C5-Pad1) -> /power/STEPIN
- Q1 pad 3: GND -> Net-(C5-Pad1)
- Q7 pad 1: Net-(C11-Pad1) -> GND
- Q7 pad 2: Net-(C8-Pad1) -> Net-(C11-Pad1)
- Q7 pad 3: GND -> Net-(C8-Pad1)
- Q8 pad 1: Net-(C12-Pad2) -> GND
- Q8 pad 2: Net-(C9-Pad1) -> Net-(C12-Pad2)
- Q8 pad 3: GND -> Net-(C9-Pad1)
Routing:
- net Net-(C11-Pad1): track 67.9 -> 30.7 mm, vias 4 -> 1
- net Net-(D16-Pad2): track 0.00 -> 36.8 mm, vias 0 -> 3
- net Net-(C12-Pad2): track 37.7 -> 34.5 mm
- net Net-(C5-Pad1): track 14.2 -> 11.1 mm
- net Net-(C9-Pad1): track 10.4 -> 7.94 mm
- net /power/STEPIN: track 61.6 -> 62.6 mm
- net GND: track 1.85 -> 2.10 mm, vias 96 -> 92

Commit message: Fix bad pins mapping on relay.
Parts:
- turned D13 to 0 degrees
Routing:
- net /RELA0: track 14.4 -> 33.1 mm, vias 0 -> 4
- net /RELA-: track 25.6 -> 11.3 mm
- net SERVO-VCC: track 65.2 -> 74.8 mm
- net /RELB0: track 20.2 -> 28.6 mm, vias 4 -> 0
- net /RELB-: track 32.9 -> 28.6 mm, vias 0 -> 4
- net /RELB+: track 20.8 -> 19.2 mm
- net GND: vias 92 -> 91

Commit message: Fix bad servo pinout.
Parts:
- moved F3 1.00 mm to (196.0, 99.9)
Connections:
- J2 pad 1: SERVO-VCC -> GND
- J2 pad 2: GND -> SERVO-VCC
Routing:
- net SERVO-VCC: track 74.8 -> 79.8 mm, vias 1 -> 2
- net /power/STEPOUT: track 3.86 -> 3.22 mm
- net GND: vias 91 -> 84
Other:
- board text added: "PWM"

Commit message: Pcb: power relay from main 5V.
Connections:
- D13 pad 1: SERVO-VCC -> VCC
- K1 pad 1: SERVO-VCC -> VCC
Routing:
- net SERVO-VCC: track 79.8 -> 49.3 mm
- net VCC: track 51.6 -> 56.7 mm
Changed lines of the file:
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@@
     (fp_line (start -1 0.6) (end 1 0.6) (layer "F.Fab") (width 0.1))
     (pad "1" smd roundrect (at -1.025 0) (size 1.15 1.4) (layers "F.Cu" "F.Paste" "F.Mask") (roundrect_rratio 0.217391)
-      (net 39 "SERVO-VCC") (pinfunction "K") (pintype "passive"))
+      (net 1 "VCC") (pinfunction "K") (pintype "passive"))
     (pad "2" smd roundrect (at 1.025 0) (size 1.15 1.4) (layers "F.Cu" "F.Paste" "F.Mask") (roundrect_rratio 0.217391)
       (net 38 "Net-(D13-Pad2)") (pinfunction "A") (pintype "passive"))
@@
     (fp_line (start 9.398 -5.08) (end -10.922 -5.08) (layer "B.Fab") (width 0.12))
     (pad "1" thru_hole circle (at -9.652 -3.81 90) (size 2 2) (drill 0.8) (layers *.Cu *.Mask)
-      (net 39 "SERVO-VCC") (pintype "passive"))
+      (net 1 "VCC") (pintype "passive"))
     (pad "3" thru_hole circle (at 8.128 -3.81 90) (size 2 2) (drill 0.8) (layers *.Cu *.Mask)
       (net 25 "/RELB-") (pintype "passive"))
@@
   (segment (start 196.088 82.55) (end 196.088 83.566) (width 0.8) (layer "F.Cu") (net 1))
   (segment (start 174.752 80.518) (end 172.339 80.518) (width 0.4) (layer "F.Cu") (net 1))
+  (segment (start 155.324 81.208) (end 155.324 79.753) (width 0.8) (layer "F.Cu") (net 1))
   (segment (start 171.934 76.732) (end 171.934 78.462) (width 0.4) (layer "F.Cu") (net 1))
   (segment (start 197.134 82.556) (end 196.094 82.556) (width 0.8) (layer "F.Cu") (net 1))
@@
   (segment (start 196.088 83.566) (end 197.124 83.566) (width 0.8) (layer "F.Cu") (net 1))
   (segment (start 170.878002 91.758) (end 170.815002 91.821) (width 0.4) (layer "F.Cu") (net 1))
+  (segment (start 157.765 77.312) (end 157.994 77.312) (width 0.8) (layer "F.Cu") (net 1))
   (segment (start 197.134 82.556) (end 197.098 82.556) (width 0.8) (layer "F.Cu") (net 1))
   (segment (start 170.887 75.192) (end 170.887 75.637) (width 0.4) (layer "F.Cu") (net 1))
@@
   (segment (start 175.387 81.153) (end 174.752 80.518) (width 0.4) (layer "F.Cu") (net 1))
   (segment (start 172.339 80.518) (end 171.934 80.113) (width 0.4) (layer "F.Cu") (net 1))
+  (segment (start 155.324 79.753) (end 157.765 77.312) (width 0.8) (layer "F.Cu") (net 1))
   (via (at 173.91 91.758) (size 0.8) (drill 0.4) (layers "F.Cu" "B.Cu") (net 1))
   (via (at 198.134 83.556) (size 0.8) (drill 0.4) (layers "F.Cu" "B.Cu") (net 1))
@@
   (segment (start 191.896 102.458) (end 193.263 102.458) (width 0.4) (layer "F.Cu") (net 39))
   (segment (start 172.286 87.758) (end 173.486 87.758) (width 0.4) (layer "F.Cu") (net 39))
-  (segment (start 155.324 81.208) (end 155.324 79.753) (width 0.8) (layer "F.Cu") (net 39))
   (segment (start 174.894 86.35) (end 174.894 86.105998) (width 0.4) (layer "F.Cu") (net 39))
-  (segment (start 157.765 77.312) (end 157.994 77.312) (width 0.8) (layer "F.Cu") (net 39))
-  (segment (start 155.324 79.753) (end 157.765 77.312) (width 0.8) (layer "F.Cu") (net 39))
   (via (at 193.263 102.458) (size 0.8) (drill 0.4) (layers "F.Cu" "B.Cu") (net 39))
   (via (at 174.894 86.105998) (size 0.8) (drill 0.4) (layers "F.Cu" "B.Cu") (net 39))
-  (segment (start 198.008 104.676081) (end 198.008 103.474) (width 0.8) (layer "B.Cu") (net 39))
-  (segment (start 197.020081 105.664) (end 198.008 104.676081) (width 0.8) (layer "B.Cu") (net 39))
+  (segment (start 198.008 104.676081) (end 198.008 103.474) (width 0.4) (layer "B.Cu") (net 39))
+  (segment (start 191.231 103.474) (end 183.657 103.474) (width 0.4) (layer "B.Cu") (net 39))
+  (segment (start 174.910001 86.121999) (end 174.894 86.105998) (width 0.8) (layer "B.Cu") (net 39))
+  (segment (start 197.020081 105.664) (end 198.008 104.676081) (width 0.4) (layer "B.Cu") (net 39))
   (segment (start 191.643 103.886) (end 191.835 103.886) (width 0.4) (layer "B.Cu") (net 39))
-  (segment (start 183.657 103.474) (end 174.910001 94.727001) (width 0.8) (layer "B.Cu") (net 39))
   (segment (start 191.231 103.474) (end 191.643 103.886) (width 0.4) (layer "B.Cu") (net 39))
   (segment (start 198.008 103.474) (end 198.008 100.4775) (width 2) (layer "B.Cu") (net 39))
-  (segment (start 174.910001 82.916001) (end 173.202 81.208) (width 0.8) (layer "B.Cu") (net 39))
-  (segment (start 173.202 81.208) (end 166.298 81.208) (width 0.8) (layer "B.Cu") (net 39))
-  (segment (start 157.665 78.867) (end 155.324 81.208) (width 0.8) (layer "B.Cu") (net 39))
   (segment (start 198.008 100.4775) (end 197.4485 99.918) (width 1.5) (layer "B.Cu") (net 39))
-  (segment (start 191.231 103.474) (end 183.657 103.474) (width 0.8) (layer "B.Cu") (net 39))
-  (segment (start 163.957 78.867) (end 157.665 78.867) (width 0.8) (layer "B.Cu") (net 39))
-  (segment (start 174.910001 94.727001) (end 174.910001 82.916001) (width 0.8) (layer "B.Cu") (net 39))
   (segment (start 191.835 103.886) (end 193.263 102.458) (width 0.4) (layer "B.Cu") (net 39))
-  (segment (start 193.421 105.664) (end 191.231 103.474) (width 0.8) (layer "B.Cu") (net 39))
-  (segment (start 193.421 105.664) (end 197.020081 105.664) (width 0.8) (layer "B.Cu") (net 39))
-  (segment (start 166.298 81.208) (end 163.957 78.867) (width 0.8) (layer "B.Cu") (net 39))
+  (segment (start 183.657 103.474) (end 174.910001 94.727001) (width 0.4) (layer "B.Cu") (net 39))
+  (segment (start 174.910001 94.727001) (end 174.910001 86.121999) (width 0.4) (layer "B.Cu") (net 39))
+  (segment (start 193.421 105.664) (end 191.231 103.474) (width 0.4) (layer "B.Cu") (net 39))
+  (segment (start 193.421 105.664) (end 197.020081 105.664) (width 0.4) (layer "B.Cu") (net 39))
   (segment (start 195.976 62.7975) (end 195.976 65.12) (width 0.8) (layer "F.Cu") (net 40))
   (segment (start 195.976 64.485) (end 195.976 65.12) (width 0.4) (layer "F.Cu") (net 40))
