File: pcb/hwexla.kicad_sch (KiCad schematic)
At the start: 32 parts, among them J1 DB25_Male, J2 Conn_01x03, J3 AVR-ISP-6, J4 Conn_01x06, SW1 SW_Push, U1 ATmega8A-AU, U2 RR112-1

Commit message: Fix errors & warnings reported by DRC.
Parts:
- H1, H2: footprint MountingHole:MountingHole_2.2mm_M2_Pad_Via -> MountingHole:MountingHole_2.2mm_M2_Pad
- U1: symbol MCU_Microchip_ATmega:ATmega328P-AU -> MCU_Microchip_ATmega:ATmega328P-A
- U2: footprint Package_TO_SOT_SMD:SOT-23 -> Package_TO_SOT_SMD:SOT-23W
Connections:
- net L-BTN-OUT: now also U1.7 (XTAL1/PB6); no longer U1.32 (PD2)
- net L-OUT-: now also U1.32 (PD2); no longer U1.7 (XTAL1/PB6)
Changed lines of the file:
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@@
-    (stroke (width 0) (type default) (color 0 0 0 0))
-  )
-  (wire (pts (xy 142.24 55.88) (xy 142.24 77.47))
     (stroke (width 0) (type default) (color 0 0 0 0))
   )
@@
     (stroke (width 0) (type default) (color 0 0 0 0))
   )
-  (wire (pts (xy 142.24 55.88) (xy 185.42 55.88))
-    (stroke (width 0) (type default) (color 0 0 0 0))
-  )
   (wire (pts (xy 73.66 67.31) (xy 40.64 67.31))
     (stroke (width 0) (type default) (color 0 0 0 0))
@@
     (stroke (width 0) (type default) (color 0 0 0 0))
   )
+  (wire (pts (xy 125.73 55.88) (xy 185.42 55.88))
+    (stroke (width 0) (type default) (color 0 0 0 0))
+  )
   (wire (pts (xy 69.85 149.86) (xy 69.85 152.4))
     (stroke (width 0) (type default) (color 0 0 0 0))
@@
     (stroke (width 0) (type default) (color 0 0 0 0))
   )
+  (wire (pts (xy 125.73 87.63) (xy 125.73 55.88))
+    (stroke (width 0) (type default) (color 0 0 0 0))
+  )
   (wire (pts (xy 173.99 86.36) (xy 185.42 86.36))
     (stroke (width 0) (type default) (color 0 0 0 0))
@@
     (stroke (width 0) (type default) (color 0 0 0 0))
   )
+  (wire (pts (xy 185.42 88.9) (xy 142.24 88.9))
+    (stroke (width 0) (type default) (color 0 0 0 0))
+  )
   (wire (pts (xy 60.96 118.11) (xy 60.96 110.49))
     (stroke (width 0) (type default) (color 0 0 0 0))
@@
     (stroke (width 0) (type default) (color 0 0 0 0))
   )
+  (wire (pts (xy 142.24 88.9) (xy 142.24 77.47))
+    (stroke (width 0) (type default) (color 0 0 0 0))
+  )
   (wire (pts (xy 125.73 107.95) (xy 111.76 107.95))
     (stroke (width 0) (type default) (color 0 0 0 0))
@@
   )
   (wire (pts (xy 40.64 102.87) (xy 43.18 102.87))
-    (stroke (width 0) (type default) (color 0 0 0 0))
-  )
-  (wire (pts (xy 125.73 88.9) (xy 185.42 88.9))
-    (stroke (width 0) (type default) (color 0 0 0 0))
-  )
-  (wire (pts (xy 125.73 87.63) (xy 125.73 88.9))
     (stroke (width 0) (type default) (color 0 0 0 0))
   )
@@
     (effects (font (size 1.27 1.27)) (justify left bottom))
   )
-  (label "L-BTN-OUT" (at 182.88 88.9 180)
+  (label "L-BTN-OUT" (at 182.88 55.88 180)
     (effects (font (size 1.27 1.27)) (justify right bottom))
   )
-  (label "L-OUT-" (at 182.88 55.88 180)
+  (label "L-OUT-" (at 182.88 88.9 180)
     (effects (font (size 1.27 1.27)) (justify right bottom))
   )
@@
     (pin "9")
   )
-  (symbol (lib_id "MCU_Microchip_ATmega:ATmega328P-AU") (at 200.66 71.12 0) (mirror y) (unit 1)
+  (symbol (lib_id "MCU_Microchip_ATmega:ATmega328P-A") (at 200.66 71.12 0) (mirror y) (unit 1)
     (in_bom yes) (on_board yes)
     (property "Reference" "U1" (id 0) (at 196.85 109.22 0))
@@
       (effects (font (size 1.27 1.27)) (justify left))
     )
-    (property "Footprint" "MountingHole:MountingHole_2.2mm_M2_Pad_Via" (id 2) (at 254 106.68 0)
+    (property "Footprint" "MountingHole:MountingHole_2.2mm_M2_Pad" (id 2) (at 254 106.68 0)
       (effects (font (size 1.27 1.27)) hide)
     )
@@
       (effects (font (size 1.27 1.27)) (justify left))
     )
-    (property "Footprint" "MountingHole:MountingHole_2.2mm_M2_Pad_Via" (id 2) (at 229.87 106.68 0)
+    (property "Footprint" "MountingHole:MountingHole_2.2mm_M2_Pad" (id 2) (at 229.87 106.68 0)
       (effects (font (size 1.27 1.27)) hide)
     )
@@
       (effects (font (size 1.27 1.27)) (justify right))
     )
-    (property "Footprint" "Package_TO_SOT_SMD:SOT-23" (id 2) (at 67.31 171.45 0)
+    (property "Footprint" "Package_TO_SOT_SMD:SOT-23W" (id 2) (at 67.31 171.45 0)
       (effects (font (size 1.27 1.27) italic) (justify left) hide)
     )
-    (property "Datasheet" "http://www.allegromicro.com/en/Products/Part_Numbers/1101/1101.pdf" (id 3) (at 67.31 146.05 0)
+    (property "Datasheet" "https://www.allegromicro.com/-/media/files/datasheets/a110x-datasheet.ashx" (id 3) (at 67.31 146.05 0)
       (effects (font (size 1.27 1.27)) hide)
     )
@@
       (effects (font (size 1.27 1.27)) (justify left) hide)
     )
-    (property "Datasheet" "https://datasheet.lcsc.com/lcsc/1810311712_onsemi-SMF05CT1G_C15879.pdf" (id 3) (at 227.965 146.685 0)
+    (property "Datasheet" "http://www.littelfuse.com/~/media/files/littelfuse/technical%20resources/documents/data%20sheets/sp05xxba.pdf" (id 3) (at 227.965 146.685 0)
       (effects (font (size 1.27 1.27)) hide)
     )
@@
       (effects (font (size 1.27 1.27)) (justify left) hide)
     )
-    (property "Datasheet" "https://datasheet.lcsc.com/lcsc/1810311712_onsemi-SMF05CT1G_C15879.pdf" (id 3) (at 130.175 169.545 0)
+    (property "Datasheet" "http://www.littelfuse.com/~/media/files/littelfuse/technical%20resources/documents/data%20sheets/sp05xxba.pdf" (id 3) (at 130.175 169.545 0)
       (effects (font (size 1.27 1.27)) hide)
     )
@@
     )
     (path "/00000000-0000-0000-0000-000061c397fd"
-      (reference "H1") (unit 1) (value "MountingHole_Pad") (footprint "MountingHole:MountingHole_2.2mm_M2_Pad_Via")
+      (reference "H1") (unit 1) (value "MountingHole_Pad") (footprint "MountingHole:MountingHole_2.2mm_M2_Pad")
     )
     (path "/00000000-0000-0000-0000-000061c39558"
-      (reference "H2") (unit 1) (value "MountingHole_Pad") (footprint "MountingHole:MountingHole_2.2mm_M2_Pad_Via")
+      (reference "H2") (unit 1) (value "MountingHole_Pad") (footprint "MountingHole:MountingHole_2.2mm_M2_Pad")
     )
     (path "/00000000-0000-0000-0000-000061a8e3f4"
@@
     )
     (path "/00000000-0000-0000-0000-000061f15c9f"
-      (reference "U2") (unit 1) (value "RR112-1") (footprint "Package_TO_SOT_SMD:SOT-23")
+      (reference "U2") (unit 1) (value "RR112-1") (footprint "Package_TO_SOT_SMD:SOT-23W")
     )
     (path "/00000000-0000-0000-0000-000061aa5240/00000000-0000-0000-0000-000061bb8ea3"

Commit message: Allow using of SOT353 TVS.
Connections:
- net MOSI: now also D4.3 (K)
- no-connect marks 7 -> 6
Other:
- note added: "Pin 3 for compatibility with SOT353"
Changed lines of the file:
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@@
   (junction (at 237.49 92.71) (diameter 0) (color 0 0 0 0)
+  )
+  (junction (at 222.25 137.16) (diameter 0) (color 0 0 0 0)
   )
   (junction (at 237.49 82.55) (diameter 0) (color 0 0 0 0)
@@
   (no_connect (at 40.64 80.01))
   (no_connect (at 135.89 167.64))
-  (no_connect (at 222.25 144.78))
   (bus_entry (at 163.83 53.34) (size 2.54 2.54)
     (stroke (width 0) (type default) (color 0 0 0 0))
@@
     (stroke (width 0) (type default) (color 0 0 0 0))
   )
+  (wire (pts (xy 222.25 137.16) (xy 227.33 137.16))
+    (stroke (width 0) (type default) (color 0 0 0 0))
+  )
   (wire (pts (xy 146.05 99.06) (xy 185.42 99.06))
     (stroke (width 0) (type default) (color 0 0 0 0))
@@
     (stroke (width 0) (type default) (color 0 0 0 0))
   )
+  (wire (pts (xy 222.25 137.16) (xy 222.25 144.78))
+    (stroke (width 0) (type default) (color 0 0 0 0))
+  )
   (wire (pts (xy 43.18 97.79) (xy 40.64 97.79))
     (stroke (width 0) (type default) (color 0 0 0 0))
@@
     (stroke (width 0) (type default) (color 0 0 0 0))
   )
-  (wire (pts (xy 210.82 137.16) (xy 227.33 137.16))
+  (wire (pts (xy 210.82 137.16) (xy 222.25 137.16))
     (stroke (width 0) (type default) (color 0 0 0 0))
   )
@@
     (stroke (width 0) (type default) (color 0 0 0 0))
   )
+  (text "Pin 3 for compatibility with SOT353" (at 229.87 156.21 0)
+    (effects (font (size 1.27 1.27)) (justify left bottom))
+  )
   (text "Variants:\nATmega328p, ATmega328pb" (at 217.17 76.2 0)

Commit message: Fix bad servo pinout.
Connections:
- net GND: now also J2.1 (Pin_1); no longer J2.2 (Pin_2)
- net SERVO-VCC: now also J2.2 (Pin_2); no longer J2.1 (Pin_1)
Changed lines of the file:
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@@
+    (stroke (width 0) (type default) (color 0 0 0 0))
+  )
+  (wire (pts (xy 147.32 48.26) (xy 147.32 63.5))
+    (stroke (width 0) (type default) (color 0 0 0 0))
+  )
+  (wire (pts (xy 60.96 110.49) (xy 73.66 110.49))
+    (stroke (width 0) (type default) (color 0 0 0 0))
+  )
+  (wire (pts (xy 43.18 74.93) (xy 40.64 74.93))
+    (stroke (width 0) (type default) (color 0 0 0 0))
+  )
+  (wire (pts (xy 40.64 95.25) (xy 45.72 95.25))
+    (stroke (width 0) (type default) (color 0 0 0 0))
+  )
+  (wire (pts (xy 146.05 111.76) (xy 146.05 115.57))
+    (stroke (width 0) (type default) (color 0 0 0 0))
+  )
+  (wire (pts (xy 45.72 110.49) (xy 58.42 110.49))
+    (stroke (width 0) (type default) (color 0 0 0 0))
+  )
+  (wire (pts (xy 166.37 55.88) (xy 185.42 55.88))
+    (stroke (width 0) (type default) (color 0 0 0 0))
+  )
+  (bus (pts (xy 163.83 66.04) (xy 163.83 68.58))
+    (stroke (width 0) (type default) (color 0 0 0 0))
+  )
+  (wire (pts (xy 73.66 97.79) (xy 66.04 97.79))
+    (stroke (width 0) (type default) (color 0 0 0 0))
+  )
+  (wire (pts (xy 43.18 113.03) (xy 43.18 118.11))
     (stroke (width 0) (type default) (color 0 0 0 0))
   )
@@
     (stroke (width 0) (type default) (color 0 0 0 0))
   )
-  (wire (pts (xy 147.32 48.26) (xy 147.32 63.5))
-    (stroke (width 0) (type default) (color 0 0 0 0))
-  )
-  (wire (pts (xy 60.96 110.49) (xy 73.66 110.49))
-    (stroke (width 0) (type default) (color 0 0 0 0))
-  )
-  (wire (pts (xy 43.18 74.93) (xy 40.64 74.93))
-    (stroke (width 0) (type default) (color 0 0 0 0))
-  )
-  (wire (pts (xy 40.64 95.25) (xy 45.72 95.25))
-    (stroke (width 0) (type default) (color 0 0 0 0))
-  )
-  (wire (pts (xy 146.05 111.76) (xy 146.05 115.57))
-    (stroke (width 0) (type default) (color 0 0 0 0))
-  )
-  (wire (pts (xy 45.72 110.49) (xy 58.42 110.49))
-    (stroke (width 0) (type default) (color 0 0 0 0))
-  )
-  (wire (pts (xy 166.37 55.88) (xy 185.42 55.88))
-    (stroke (width 0) (type default) (color 0 0 0 0))
-  )
-  (bus (pts (xy 163.83 66.04) (xy 163.83 68.58))
-    (stroke (width 0) (type default) (color 0 0 0 0))
-  )
-  (wire (pts (xy 73.66 97.79) (xy 66.04 97.79))
-    (stroke (width 0) (type default) (color 0 0 0 0))
-  )
-  (wire (pts (xy 43.18 113.03) (xy 43.18 118.11))
-    (stroke (width 0) (type default) (color 0 0 0 0))
-  )
   (wire (pts (xy 215.9 142.24) (xy 219.71 142.24))
     (stroke (width 0) (type default) (color 0 0 0 0))
@@
     (stroke (width 0) (type default) (color 0 0 0 0))
   )
-  (wire (pts (xy 257.81 87.63) (xy 255.27 87.63))
-    (stroke (width 0) (type default) (color 0 0 0 0))
-  )
   (wire (pts (xy 73.66 62.23) (xy 40.64 62.23))
     (stroke (width 0) (type default) (color 0 0 0 0))
@@
     (stroke (width 0) (type default) (color 0 0 0 0))
   )
+  (wire (pts (xy 257.81 87.63) (xy 252.73 87.63))
+    (stroke (width 0) (type default) (color 0 0 0 0))
+  )
   (wire (pts (xy 111.76 87.63) (xy 127 87.63))
     (stroke (width 0) (type default) (color 0 0 0 0))
@@
     (stroke (width 0) (type default) (color 0 0 0 0))
   )
-  (wire (pts (xy 255.27 95.25) (xy 255.27 90.17))
+  (wire (pts (xy 252.73 87.63) (xy 252.73 95.25))
     (stroke (width 0) (type default) (color 0 0 0 0))
   )
@@
     (stroke (width 0) (type default) (color 0 0 0 0))
   )
-  (wire (pts (xy 255.27 82.55) (xy 255.27 87.63))
+  (wire (pts (xy 255.27 82.55) (xy 255.27 90.17))
     (stroke (width 0) (type default) (color 0 0 0 0))
   )
@@
     (pin "1")
   )
-  (symbol (lib_id "power:GND") (at 255.27 95.25 0) (unit 1)
-    (in_bom yes) (on_board yes)
-    (property "Reference" "#PWR09" (id 0) (at 255.27 101.6 0)
-      (effects (font (size 1.27 1.27)) hide)
-    )
-    (property "Value" "GND" (id 1) (at 255.397 99.6442 0))
-    (property "Footprint" "" (id 2) (at 255.27 95.25 0)
-      (effects (font (size 1.27 1.27)) hide)
-    )
-    (property "Datasheet" "" (id 3) (at 255.27 95.25 0)
-      (effects (font (size 1.27 1.27)) hide)
-    )
+  (symbol (lib_id "power:GND") (at 252.73 95.25 0) (unit 1)
+    (in_bom yes) (on_board yes)
+    (property "Reference" "#PWR09" (id 0) (at 252.73 101.6 0)
+      (effects (font (size 1.27 1.27)) hide)
+    )
+    (property "Value" "GND" (id 1) (at 252.857 99.6442 0))
+    (property "Footprint" "" (id 2) (at 252.73 95.25 0)
+      (effects (font (size 1.27 1.27)) hide)
+    )
+    (property "Datasheet" "" (id 3) (at 252.73 95.25 0)
+      (effects (font (size 1.27 1.27)) hide)
+    )

Commit message: Pcb: power relay from main 5V.
Changed lines of the file:
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@@
   (junction (at 200.66 26.67) (diameter 0) (color 0 0 0 0)
   )
-  (junction (at 113.03 39.37) (diameter 0) (color 0 0 0 0)
-  )
   (junction (at 45.72 101.6) (diameter 0) (color 0 0 0 0)
   )
@@
   (junction (at 133.35 160.02) (diameter 0) (color 0 0 0 0)
   )
-  (junction (at 113.03 48.26) (diameter 0) (color 0 0 0 0)
+  (junction (at 120.65 39.37) (diameter 0) (color 0 0 0 0)
   )
   (junction (at 227.33 137.16) (diameter 0) (color 0 0 0 0)
@@
     (stroke (width 0) (type default) (color 0 0 0 0))
   )
+  (wire (pts (xy 115.57 100.33) (xy 115.57 97.79))
+    (stroke (width 0) (type default) (color 0 0 0 0))
+  )
   (wire (pts (xy 146.05 99.06) (xy 185.42 99.06))
     (stroke (width 0) (type default) (color 0 0 0 0))
@@
     (stroke (width 0) (type default) (color 0 0 0 0))
   )
-  (wire (pts (xy 113.03 48.26) (xy 147.32 48.26))
-    (stroke (width 0) (type default) (color 0 0 0 0))
-  )
   (bus (pts (xy 163.83 52.07) (xy 163.83 53.34))
     (stroke (width 0) (type default) (color 0 0 0 0))
@@
     (stroke (width 0) (type default) (color 0 0 0 0))
   )
-  (wire (pts (xy 113.03 39.37) (xy 113.03 48.26))
-    (stroke (width 0) (type default) (color 0 0 0 0))
-  )
   (wire (pts (xy 135.89 96.52) (xy 185.42 96.52))
     (stroke (width 0) (type default) (color 0 0 0 0))
   )
-  (wire (pts (xy 113.03 39.37) (xy 123.19 39.37))
+  (wire (pts (xy 111.76 39.37) (xy 120.65 39.37))
     (stroke (width 0) (type default) (color 0 0 0 0))
   )
@@
     (stroke (width 0) (type default) (color 0 0 0 0))
   )
-  (wire (pts (xy 113.03 48.26) (xy 113.03 100.33))
-    (stroke (width 0) (type default) (color 0 0 0 0))
-  )
   (wire (pts (xy 45.72 101.6) (xy 45.72 100.33))
     (stroke (width 0) (type default) (color 0 0 0 0))
@@
     (stroke (width 0) (type default) (color 0 0 0 0))
   )
-  (wire (pts (xy 111.76 100.33) (xy 113.03 100.33))
+  (wire (pts (xy 111.76 100.33) (xy 115.57 100.33))
     (stroke (width 0) (type default) (color 0 0 0 0))
   )
@@
     (stroke (width 0) (type default) (color 0 0 0 0))
   )
-  (wire (pts (xy 111.76 39.37) (xy 113.03 39.37))
-    (stroke (width 0) (type default) (color 0 0 0 0))
-  )
   (wire (pts (xy 173.99 120.65) (xy 173.99 123.19))
     (stroke (width 0) (type default) (color 0 0 0 0))
@@
     (stroke (width 0) (type default) (color 0 0 0 0))
   )
+  (wire (pts (xy 120.65 48.26) (xy 147.32 48.26))
+    (stroke (width 0) (type default) (color 0 0 0 0))
+  )
   (wire (pts (xy 173.99 83.82) (xy 185.42 83.82))
     (stroke (width 0) (type default) (color 0 0 0 0))
   )
+  (wire (pts (xy 120.65 39.37) (xy 123.19 39.37))
+    (stroke (width 0) (type default) (color 0 0 0 0))
+  )
   (wire (pts (xy 227.33 144.78) (xy 227.33 137.16))
     (stroke (width 0) (type default) (color 0 0 0 0))
@@
   )
   (wire (pts (xy 219.71 142.24) (xy 241.3 142.24))
+    (stroke (width 0) (type default) (color 0 0 0 0))
+  )
+  (wire (pts (xy 120.65 39.37) (xy 120.65 48.26))
     (stroke (width 0) (type default) (color 0 0 0 0))
   )
@@
     (pin "6")
   )
+  (symbol (lib_id "power:VCC") (at 115.57 97.79 0) (unit 1)
+    (in_bom yes) (on_board yes)
+    (property "Reference" "#PWR?" (id 0) (at 115.57 101.6 0)
+      (effects (font (size 1.27 1.27)) hide)
+    )
+    (property "Value" "VCC" (id 1) (at 115.951 93.3958 0))
+    (property "Footprint" "" (id 2) (at 115.57 97.79 0)
+      (effects (font (size 1.27 1.27)) hide)
+    )
+    (property "Datasheet" "" (id 3) (at 115.57 97.79 0)
+      (effects (font (size 1.27 1.27)) hide)
+    )
+    (pin "1")
+  )
   (sheet (at 73.66 33.02) (size 38.1 12.7) (fields_autoplaced)
     (stroke (width 0) (type solid) (color 0 0 0 0))
@@
       (reference "#PWR048") (unit 1) (value "GND") (footprint "")
     )
+    (path "/63183de5-2468-46f3-bb84-63dadb2b103e"
+      (reference "#PWR?") (unit 1) (value "VCC") (footprint "")
+    )
     (path "/00000000-0000-0000-0000-000061d6e7e0"
