File: pcb/hwexla.kicad_sch (KiCad schematic)
At the start: 34 parts, among them J1 DB25_Male, J2 Conn_01x03, J3 AVR-ISP-6, J4 Conn_01x06, SW1 SW_Push, U1 ATmega8A-AU, U2 RR112-1

Commit message: Move F3 so it is not under connector.
Parts:
- TP2: footprint TestPoint:TestPoint_Loop_D3.50mm_Drill1.4mm_Beaded -> TestPoint:TestPoint_Loop_D1.80mm_Drill1.0mm_Beaded
Changed lines of the file:
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@@
       (effects (font (size 1.27 1.27)) (justify left))
     )
-    (property "Footprint" "TestPoint:TestPoint_Loop_D3.50mm_Drill1.4mm_Beaded" (at 264.16 41.91 0)
+    (property "Footprint" "TestPoint:TestPoint_Loop_D1.80mm_Drill1.0mm_Beaded" (at 264.16 41.91 0)
       (effects (font (size 1.27 1.27)) hide)
     )

Commit message: Use more proper footprint for SMD button.
Parts:
- SW1: footprint Button_Switch_SMD:SW_Push_1P1T_NO_6x6mm_H9.5mm -> Button_Switch_SMD:SW_SPST_Omron_B3FS-100xP
Changed lines of the file:
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@@
       (effects (font (size 1.27 1.27)) (justify right))
     )
-    (property "Footprint" "Button_Switch_SMD:SW_Push_1P1T_NO_6x6mm_H9.5mm" (at 179.07 128.27 0)
+    (property "Footprint" "Button_Switch_SMD:SW_SPST_Omron_B3FS-100xP" (at 179.07 128.27 0)
       (effects (font (size 1.27 1.27)) hide)
     )

Commit message: Use 10k for green LED.
Parts:
- R3: value 1k -> 10k; LCSC C17513 -> C17414
Changed lines of the file:
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@@
       (effects (font (size 1.27 1.27)) (justify left))
     )
-    (property "Value" "1k" (at 134.112 109.093 0)
+    (property "Value" "10k" (at 134.112 109.093 0)
       (effects (font (size 1.27 1.27)) (justify left))
     )
@@
       (effects (font (size 1.27 1.27)) hide)
     )
-    (property "LCSC" "C17513" (at 135.89 107.95 0)
+    (property "LCSC" "C17414" (at 135.89 107.95 0)
       (effects (font (size 1.27 1.27)) hide)
     )

Commit message: Add protection on internal inputs, divide stepdown voltage measuring by 2.
Parts:
- added C15: 100p, Capacitor_SMD:C_0805_2012Metric_Pad1.18x1.45mm_HandSolder, symbol Device:C
- added R15, R16: 10k, Resistor_SMD:R_0805_2012Metric_Pad1.20x1.40mm_HandSolder, symbol Device:R
- H1: value MountingHole_Pad -> ServoMount1
- H2: value MountingHole_Pad -> ServoMount2
- H3, H4: value MountingHole -> JLCPCB
- J1: symbol Connector:DB25_Male -> Connector:DB25_Plug
Connections:
- net GND: now also C15.2, R16.2
- net SERVO-VCC: now also R15.1; no longer U1.23 (PC0)
- new net L-SERVO-VCC: C15.1, R15.2, R16.1, U1.23 (PC0)
Other:
- note added: "SERVO"
- moved on the sheet: C1, C13, C2, C3, C4, D1, D2, D3, D4, F1, H1, H2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

Commit message: Change C15 to 100n.
Parts:
- C15: value 100p -> 100n; LCSC C1790 -> C49678
Changed lines of the file:
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@@
       (effects (font (size 1.27 1.27)) (justify left))
     )
-    (property "Value" "100p" (at 150.749 75.438 0)
+    (property "Value" "100n" (at 150.749 75.438 0)
       (effects (font (size 1.27 1.27)) (justify left))
     )
@@
       (effects (font (size 1.27 1.27)) hide)
     )
-    (property "LCSC" "C1790" (at 153.67 74.295 0)
+    (property "LCSC" "C49678" (at 153.67 74.295 0)
       (effects (font (size 1.27 1.27)) hide)
     )
