File: pcb/hwexla.kicad_sch (KiCad schematic)
At the start: 37 parts, among them J1 DB25_Male, J2 Conn_01x03, J3 AVR-ISP-6, J4 Conn_01x06, SW1 SW_Push, U1 ATmega8A-AU, U2 RR112-1

Commit message: Sch: use JLCPCB tooling holes from MountingHole lib.
Parts:
- H3, H4: footprint jlcpcb_tooling_holes:jlcpcb_tooling_holes -> MountingHole:ToolingHole_1.152mm
Changed lines of the file:
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@@
 			)
 		)
-		(property "Footprint" "jlcpcb_tooling_holes:jlcpcb_tooling_holes"
+		(property "Footprint" "MountingHole:ToolingHole_1.152mm"
 			(at 36.195 189.865 0)
 			(effects
@@
 			)
 		)
-		(property "Footprint" "jlcpcb_tooling_holes:jlcpcb_tooling_holes"
+		(property "Footprint" "MountingHole:ToolingHole_1.152mm"
 			(at 36.195 184.15 0)
 			(effects

Commit message: Add TME part numbers.
Parts:
- J3: TME (none) -> ZL262-6DG
- J4: TME (none) -> ZL262-6SG
- SW1: TME (none) -> TSS62N
- U2: ValueAlt (none) -> CT8150PC-IS3
Changed lines of the file:
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@@
 			)
 		)
-		(property "Datasheet" " ~"
+		(property "Datasheet" "~"
 			(at 292.1 156.21 0)
 			(effects
@@
 				)
 				(hide yes)
+			)
+		)
+		(property "TME" "ZL262-6DG"
+			(at 259.08 160.02 0)
+			(show_name yes)
+			(effects
+				(font
+					(size 1.27 1.27)
+				)
 			)
 		)
@@
 			)
 		)
+		(property "TME" "TSS62N"
+			(at 182.88 133.35 90)
+			(show_name yes)
+			(effects
+				(font
+					(size 1.27 1.27)
+				)
+			)
+		)
 		(pin "1"
 		)
@@
 			)
 		)
+		(property "TME" "ZL262-6SG"
+			(at 152.4 180.34 0)
+			(show_name yes)
+			(effects
+				(font
+					(size 1.27 1.27)
+				)
+			)
+		)
 		(pin "1"
 		)
@@
 			)
 		)
+		(property "ValueAlt" "CT8150PC-IS3"
+			(at 27.94 170.18 0)
+			(show_name yes)
+			(effects
+				(font
+					(size 1.27 1.27)
+				)
+			)
+		)

Commit message: Fix DRC issues.
Connections:
- net MOSI: no longer D4.3 (K)
- no-connect marks 6 -> 7
Other:
- note removed: "Pin 3 for compatibility with SOT353"
Changed lines of the file:
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@@
 		(comment 4 "Released under the Creative Commons Attribution-ShareAlike 4.0 License")
-	)
-	(text "Pin 3 for compatibility with SOT353"
-		(exclude_from_sim no)
-		(at 230.505 158.75 0)
-		(effects
-			(font
-				(size 1.27 1.27)
-			)
-			(justify right bottom)
-		)
 	)
 	(text "Variants:\nATmega8a, ATmega328p, ATmega328pb"
@@
 	)
 	(junction
-		(at 238.125 139.7)
-		(diameter 0)
-		(color 0 0 0 0)
-	)
-	(junction
 		(at 133.35 160.02)
 		(diameter 0)
@@
 		(at 135.89 167.64)
 	)
+	(no_connect
+		(at 238.125 147.32)
+	)
 	(bus_entry
 		(at 162.56 58.42)
@@
 	(wire
 		(pts
-			(xy 238.125 139.7) (xy 233.045 139.7)
+			(xy 233.045 139.7) (xy 249.555 139.7)
 		)
 		(stroke
@@
 	(wire
 		(pts
-			(xy 238.125 139.7) (xy 238.125 147.32)
-		)
-		(stroke
-			(width 0)
-			(type default)
-		)
-	)
-	(wire
-		(pts
 			(xy 41.91 102.87) (xy 39.37 102.87)
 		)
@@
 		)
 		(stroke
-			(width 0)
-			(type default)
-		)
-	)
-	(wire
-		(pts
-			(xy 249.555 139.7) (xy 238.125 139.7)
-		)
-		(stroke

Commit message: Bridge both program&debug power solderjumpers.
Parts:
- JP1, JP2: value SolderJumper_2_Open -> ~; footprint Jumper:SolderJumper-2_P1.3mm_Open_RoundedPad1.0x1.5mm -> Jumper:SolderJumper-2_P1.3mm_Bridged_RoundedPad1.0x1.5mm; symbol Jumper:SolderJumper_2_Open -> Jumper:SolderJumper_2_Bridged; now left out of the parts list
Changed lines of the file:
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@@
 	)
 	(symbol
-		(lib_id "Jumper:SolderJumper_2_Open")
+		(lib_id "Jumper:SolderJumper_2_Bridged")
 		(at 114.3 165.1 0)
 		(unit 1)
 		(exclude_from_sim no)
-		(in_bom yes)
+		(in_bom no)
 		(on_board yes)
 		(dnp no)
 		(property "Reference" "JP2"
-			(at 114.3 170.18 0)
-			(effects
-				(font
-					(size 1.27 1.27)
-				)
-			)
-		)
-		(property "Value" "SolderJumper_2_Open"
+			(at 114.3 168.275 0)
+			(effects
+				(font
+					(size 1.27 1.27)
+				)
+			)
+		)
+		(property "Value" "~"
 			(at 114.3 167.64 0)
 			(effects
@@
 			)
 		)
-		(property "Footprint" "Jumper:SolderJumper-2_P1.3mm_Open_RoundedPad1.0x1.5mm"
+		(property "Footprint" "Jumper:SolderJumper-2_P1.3mm_Bridged_RoundedPad1.0x1.5mm"
 			(at 114.3 165.1 0)
 			(effects
@@
 			)
 		)
-		(property "Description" ""
+		(property "Description" "Solder Jumper, 2-pole, closed/bridged"
 			(at 114.3 165.1 0)
 			(effects
@@
 					(size 1.27 1.27)
 				)
+				(hide yes)
 			)
 		)
@@
 	)
 	(symbol
-		(lib_id "Jumper:SolderJumper_2_Open")
+		(lib_id "Jumper:SolderJumper_2_Bridged")
 		(at 255.905 127 0)
 		(mirror y)
 		(unit 1)
 		(exclude_from_sim no)
-		(in_bom yes)
+		(in_bom no)
 		(on_board yes)
 		(dnp no)
 		(property "Reference" "JP1"
-			(at 255.905 121.793 0)
-			(effects
-				(font
-					(size 1.27 1.27)
-				)
-			)
-		)
-		(property "Value" "SolderJumper_2_Open"
+			(at 255.905 124.46 0)
+			(effects
+				(font
+					(size 1.27 1.27)
+				)
+			)
+		)
+		(property "Value" "~"
 			(at 255.905 124.1044 0)
 			(effects
@@
 			)
 		)
-		(property "Footprint" "Jumper:SolderJumper-2_P1.3mm_Open_RoundedPad1.0x1.5mm"
+		(property "Footprint" "Jumper:SolderJumper-2_P1.3mm_Bridged_RoundedPad1.0x1.5mm"
 			(at 255.905 127 0)
 			(effects
@@
 			)
 		)
-		(property "Description" ""
+		(property "Description" "Solder Jumper, 2-pole, closed/bridged"
 			(at 255.905 127 0)
 			(effects
@@
 					(size 1.27 1.27)
 				)
-			)
-		)
+				(hide yes)
+			)
+		)

Commit message: REL: fix bad wire names.
Connections:
- net RELA+: now also J1.24 (P24), J1.25 (P25); no longer J1.20 (P20), J1.21 (P21)
- net RELA-: now also J1.20 (P20), J1.21 (P21); no longer J1.24 (P24), J1.25 (P25)
- net RELB+: now also J1.8, J1.9; no longer J1.12, J1.13
- net RELB-: now also J1.12, J1.13; no longer J1.8, J1.9
Changed lines of the file:
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@@
 	(wire
 		(pts
-			(xy 59.69 115.57) (xy 72.39 115.57)
-		)
-		(stroke
-			(width 0)
-			(type default)
-		)
-	)
-	(wire
-		(pts
 			(xy 41.91 80.01) (xy 39.37 80.01)
 		)
@@
 	(wire
 		(pts
-			(xy 41.91 123.19) (xy 59.69 123.19)
+			(xy 41.91 123.19) (xy 72.39 123.19)
 		)
 		(stroke
@@
 	(wire
 		(pts
+			(xy 62.23 115.57) (xy 72.39 115.57)
+		)
+		(stroke
+			(width 0)
+			(type default)
+		)
+	)
+	(wire
+		(pts
 			(xy 262.255 129.54) (xy 262.255 127)
 		)
@@
 	(wire
 		(pts
-			(xy 62.23 102.87) (xy 62.23 123.19)
+			(xy 62.23 102.87) (xy 62.23 115.57)
 		)
 		(stroke
@@
 	(wire
 		(pts
-			(xy 59.69 123.19) (xy 59.69 115.57)
-		)
-		(stroke
-			(width 0)
-			(type default)
-		)
-	)
-	(wire
-		(pts
 			(xy 235.585 147.32) (xy 235.585 137.16)
 		)
@@
 	(wire
 		(pts
-			(xy 62.23 123.19) (xy 72.39 123.19)
-		)
-		(stroke
-			(width 0)
-			(type default)
-		)
-	)
-	(wire
-		(pts
 			(xy 72.39 82.55) (xy 39.37 82.55)
 		)
@@
 		)
 	)
-	(label "RELA+"
+	(label "RELA-"
 		(at 46.99 100.33 0)
 		(effects
@@
 		)
 	)
-	(label "RELB+"
+	(label "RELB-"
 		(at 46.99 123.19 0)
 		(effects
@@
 		)
 	)
-	(label "RELB-"
+	(label "RELB+"
 		(at 46.99 102.87 0)
 		(effects
@@
 		)
 	)
-	(label "RELA-"
+	(label "RELA+"
 		(at 46.99 115.57 0)
 		(effects
@@
 		)
 		(pin "RELA+" bidirectional
-			(at 72.39 102.87 180)
+			(at 72.39 110.49 180)
 			(effects
 				(font
@@
 		)
 		(pin "RELA-" bidirectional
-			(at 72.39 110.49 180)
+			(at 72.39 102.87 180)
 			(effects
 				(font
