File: pcb/power.kicad_sch (KiCad schematic)
At the start: 14 parts, among them J5 Conn_01x04, Q1 BT148, U3 KA78M05_TO252

Commit message: Use 2920 package for polyfuse.
Parts:
- F2: footprint Fuse:Fuse_1206_3216Metric_Pad1.42x1.75mm_HandSolder -> Fuse:Fuse_2920_7451Metric; LCSC C910830 -> C3020148
Changed lines of the file:
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@@
       (effects (font (size 1.27 1.27)))
     )
-    (property "Footprint" "Fuse:Fuse_1206_3216Metric_Pad1.42x1.75mm_HandSolder" (at 39.37 60.96 0)
+    (property "Footprint" "Fuse:Fuse_2920_7451Metric" (at 39.37 60.96 0)
       (effects (font (size 1.27 1.27)) (justify left) hide)
     )
@@
       (effects (font (size 1.27 1.27)) hide)
     )
-    (property "LCSC" "C910830" (at 44.45 59.69 0)
+    (property "LCSC" "C3020148" (at 44.45 59.69 0)
       (effects (font (size 1.27 1.27)) hide)
     )

Commit message: Decreases fuses values 1A -> 0.5A.
Servo does not need such a big current and PTC takes some time to switch
off. It's better to switch off in shorter time.
Parts:
- F2: value 1A/1.8A -> 0.5A/1A; LCSC C3020148 -> C2760297
- F3: value 1A -> 500mA; LCSC C182974 -> C3161978
Other:
- note added: "SG90 consumes 350 mA in peak according to https://protosupplies.com/product/servo-motor-micro-sg90/ Measured max current by JH: 150 mA"
- note added: "TME BSMD1206-SS0.5"
- note added: "TME SL050-60"
Changed lines of the file:
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@@
     (stroke (width 0) (type default))
+  )
+  (text "   TME\nSL050-60" (at 39.37 51.435 0)
+    (effects (font (size 1.27 1.27)) (justify left bottom))
   )
   (text "Power for servo & relay" (at 142.24 33.02 0)
     (effects (font (size 2.54 2.54)) (justify left bottom))
   )
+  (text "SG90 consumes 350 mA in peak according to\nhttps://protosupplies.com/product/servo-motor-micro-sg90/\nMeasured max current by JH: 150 mA"
+    (at 182.88 71.12 0)
+    (effects (font (size 1.27 1.27)) (justify left bottom))
+  )
   (text "External stepdown" (at 156.21 36.83 0)
     (effects (font (size 1.27 1.27)) (justify left bottom))
@@
     (effects (font (size 1.27 1.27)) (justify left bottom))
   )
+  (text "       TME\nBSMD1206-SS0.5" (at 203.835 52.07 0)
+    (effects (font (size 1.27 1.27)) (justify left bottom))
+  )
   (label "GND" (at 166.37 46.99 270) (fields_autoplaced)
     (effects (font (size 1.27 1.27)) (justify right bottom))
@@
       (effects (font (size 1.27 1.27)))
     )
-    (property "Value" "1A" (at 212.09 56.9976 90)
+    (property "Value" "500mA" (at 212.09 56.9976 90)
       (effects (font (size 1.27 1.27)))
     )
@@
       (effects (font (size 1.27 1.27)) hide)
     )
-    (property "LCSC" "C182974" (at 212.09 59.69 0)
+    (property "LCSC" "C3161978" (at 212.09 59.69 0)
       (effects (font (size 1.27 1.27)) hide)
     )
@@
       (effects (font (size 1.27 1.27)))
     )
-    (property "Value" "1A/1.8A" (at 44.45 56.2864 90)
+    (property "Value" "0.5A/1A" (at 44.45 56.2864 90)
       (effects (font (size 1.27 1.27)))
     )
@@
       (effects (font (size 1.27 1.27)) hide)
     )
-    (property "LCSC" "C3020148" (at 44.45 59.69 0)
-      (effects (font (size 1.27 1.27)) hide)
-    )
+    (property "LCSC" "C2760297" (at 44.45 59.69 0)
+      (effects (font (size 1.27 1.27)) hide)
+    )

Commit message: Add protection on internal inputs, divide stepdown voltage measuring by 2.
Parts:
- added R14: 1k, Resistor_SMD:R_0805_2012Metric_Pad1.20x1.40mm_HandSolder, symbol Device:R
Connections:
- net SERVO-POWER-EN: now also R14.1; no longer J5.1 (Pin_1), R9.1
- new net: J5.1 (Pin_1), R14.2, R9.1
Other:
- moved on the sheet: Q1
Changed lines of the file:
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@@
     (stroke (width 0) (type default))
   )
-  (wire (pts (xy 86.36 67.31) (xy 86.36 82.55))
+  (wire (pts (xy 86.36 68.58) (xy 86.36 82.55))
     (stroke (width 0) (type default))
   )
@@
     (stroke (width 0) (type default))
   )
+  (wire (pts (xy 86.36 60.96) (xy 86.36 59.69))
+    (stroke (width 0) (type default))
+  )
   (wire (pts (xy 166.37 46.99) (xy 166.37 80.01))
     (stroke (width 0) (type default))
@@
     (stroke (width 0) (type default))
   )
+  (wire (pts (xy 148.59 64.77) (xy 161.29 64.77))
+    (stroke (width 0) (type default))
+  )
   (wire (pts (xy 59.69 82.55) (xy 69.85 82.55))
     (stroke (width 0) (type default))
@@
     (stroke (width 0) (type default))
   )
-  (wire (pts (xy 157.48 64.77) (xy 161.29 64.77))
-    (stroke (width 0) (type default))
-  )
-  (wire (pts (xy 82.55 67.31) (xy 82.55 66.04))
+  (wire (pts (xy 130.175 64.77) (xy 140.97 64.77))
     (stroke (width 0) (type default))
   )
@@
     (effects (font (size 1.27 1.27)) (justify left))
   )
-  (hierarchical_label "SERVO-POWER-EN" (shape input) (at 157.48 64.77 180) (fields_autoplaced)
+  (hierarchical_label "SERVO-POWER-EN" (shape input) (at 130.175 64.77 180) (fields_autoplaced)
     (effects (font (size 1.27 1.27)) (justify right))
   )
@@
     )
   )
-  (symbol (lib_id "Device:Q_SCR_KAG") (at 86.36 63.5 0) (unit 1)
-    (in_bom yes) (on_board yes) (dnp no)
-    (property "Reference" "Q1" (at 88.5952 62.3316 0)
-      (effects (font (size 1.27 1.27)) (justify left))
-    )
-    (property "Value" "BT148" (at 88.5952 64.643 0)
-      (effects (font (size 1.27 1.27)) (justify left))
-    )
-    (property "Footprint" "Package_TO_SOT_SMD:SOT-223" (at 86.36 63.5 90)
-      (effects (font (size 1.27 1.27)) hide)
-    )
-    (property "Datasheet" "~" (at 86.36 63.5 90)
-      (effects (font (size 1.27 1.27)) hide)
-    )
-    (property "LCSC" "C256433" (at 86.36 63.5 0)
+  (symbol (lib_id "Device:Q_SCR_KAG") (at 86.36 64.77 0) (unit 1)
+    (in_bom yes) (on_board yes) (dnp no)
+    (property "Reference" "Q1" (at 88.5952 63.6016 0)
+      (effects (font (size 1.27 1.27)) (justify left))
+    )
+    (property "Value" "BT148" (at 88.5952 65.913 0)
+      (effects (font (size 1.27 1.27)) (justify left))
+    )
+    (property "Footprint" "Package_TO_SOT_SMD:SOT-223" (at 86.36 64.77 90)
+      (effects (font (size 1.27 1.27)) hide)
+    )
+    (property "Datasheet" "~" (at 86.36 64.77 90)
+      (effects (font (size 1.27 1.27)) hide)
+    )
+    (property "LCSC" "C256433" (at 86.36 64.77 0)
       (effects (font (size 1.27 1.27)) hide)
     )
@@
       (effects (font (size 1.27 1.27)) hide)
     )
+    (property "Sim.Device" "D" (at 50.8 63.5 0)
+      (effects (font (size 1.27 1.27)) hide)
+    )
+    (property "Sim.Pins" "1=K 2=A" (at 50.8 63.5 0)
+      (effects (font (size 1.27 1.27)) hide)
+    )
     (pin "1")
     (pin "2")
@@
       (effects (font (size 1.27 1.27)) hide)
     )
+    (property "Sim.Device" "D" (at 123.19 118.11 0)
+      (effects (font (size 1.27 1.27)) hide)
+    )
+    (property "Sim.Pins" "1=K 2=A" (at 123.19 118.11 0)
+      (effects (font (size 1.27 1.27)) hide)
+    )
     (pin "1")
     (pin "2")
@@
         )
       )
+    )
+  )
+  (symbol (lib_id "Device:R") (at 144.78 64.77 90) (mirror x) (unit 1)
+    (in_bom yes) (on_board yes) (dnp no)
+    (property "Reference" "R14" (at 144.78 69.9303 90)
+      (effects (font (size 1.27 1.27)))
+    )
+    (property "Value" "1k" (at 144.78 67.5061 90)
+      (effects (font (size 1.27 1.27)))
+    )
+    (property "Footprint" "Resistor_SMD:R_0805_2012Metric_Pad1.20x1.40mm_HandSolder" (at 144.78 62.992 90)
+      (effects (font (size 1.27 1.27)) hide)
+    )
+    (property "Datasheet" "~" (at 144.78 64.77 0)
+      (effects (font (size 1.27 1.27)) hide)
+    )
+    (property "LCSC" "C17513" (at 144.78 64.77 0)
+      (effects (font (size 1.27 1.27)) hide)
+    )
+    (pin "1")
+    (pin "2")
+    (instances
+      (project "hwexla"
+        (path "/1cc5480b-56b7-4379-98e2-ccafc88911a7/00000000-0000-0000-0000-000061aa561a"
+          (reference "R14") (unit 1)
+        )
+        (path "/1cc5480b-56b7-4379-98e2-ccafc88911a7/00000000-0000-0000-0000-000061aa5240"
+          (reference "R17") (unit 1)
+        )
+      )

Commit message: Upgrade to KiCad 9.
Parts:
- renumbered R14 to R17
