File: pcb/power.kicad_sch (KiCad schematic)
At the start: 15 parts, among them J5 Conn_01x04, Q1 BT148, U3 KA78M05_TO252

Commit message: Add TME part numbers as part attributes.
Parts:
- F2: TME (none) -> SL050-60
- F3: TME (none) -> BSMD1206-SS0.5
Other:
- note removed: "TME BSMD1206-SS0.5"
- note removed: "TME SL050-60"
Changed lines of the file:
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@@
 		(comment 4 "Released under the Creative Commons Attribution-ShareAlike 4.0 License")
-	)
-	(text "   TME\nSL050-60"
-		(exclude_from_sim no)
-		(at 39.37 51.435 0)
-		(effects
-			(font
-				(size 1.27 1.27)
-			)
-			(justify left bottom)
-		)
 	)
 	(text "Power for servo & relay"
@@
 		(exclude_from_sim no)
 		(at 156.21 39.37 0)
-		(effects
-			(font
-				(size 1.27 1.27)
-			)
-			(justify left bottom)
-		)
-	)
-	(text "       TME\nBSMD1206-SS0.5"
-		(exclude_from_sim no)
-		(at 203.835 52.07 0)
 		(effects
 			(font
@@
 			)
 		)
+		(property "TME" "BSMD1206-SS0.5"
+			(at 212.09 52.07 90)
+			(show_name yes)
+			(effects
+				(font
+					(size 1.27 1.27)
+				)
+			)
+		)
 		(pin "1"
 		)
@@
 			)
 		)
+		(property "TME" "SL050-60"
+			(at 44.45 50.8 90)
+			(show_name yes)
+			(effects
+				(font
+					(size 1.27 1.27)
+				)
+			)
+		)

Commit message: Add 7805 protective diode.
Parts:
- added D9: 1N5819, Diode_SMD:D_SOD-123, symbol Device:D_Schottky
- D7: value 1N4007 -> 1N5819; symbol Diode:1N4007 -> Diode:1N5819; LCSC C64898 -> C191023
Connections:
- net VCC: now also D9.2 (A)
- net at C6.1, D7.1 (K), U3.1 (VI): now also D9.1 (K)
Changed lines of the file:
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@@
 	(text "Power for logic"
 		(exclude_from_sim no)
-		(at 149.86 107.95 0)
+		(at 165.1 145.415 0)
 		(effects
 			(font
 				(size 2.54 2.54)
 			)
-			(justify left bottom)
+			(justify bottom)
 		)
 	)
@@
 	)
 	(junction
+		(at 152.4 118.11)
+		(diameter 0)
+		(color 0 0 0 0)
+	)
+	(junction
 		(at 69.85 59.69)
 		(diameter 0)
@@
 	)
 	(junction
+		(at 178.435 118.11)
+		(diameter 0)
+		(color 0 0 0 0)
+	)
+	(junction
 		(at 77.47 82.55)
 		(diameter 0)
@@
 	(wire
 		(pts
+			(xy 168.91 105.41) (xy 178.435 105.41)
+		)
+		(stroke
+			(width 0)
+			(type default)
+		)
+	)
+	(wire
+		(pts
+			(xy 178.435 118.11) (xy 185.42 118.11)
+		)
+		(stroke
+			(width 0)
+			(type default)
+		)
+	)
+	(wire
+		(pts
 			(xy 40.64 59.69) (xy 36.83 59.69)
 		)
@@
 	(wire
 		(pts
+			(xy 178.435 105.41) (xy 178.435 118.11)
+		)
+		(stroke
+			(width 0)
+			(type default)
+		)
+	)
+	(wire
+		(pts
 			(xy 86.36 59.69) (xy 100.33 59.69)
 		)
@@
 	(wire
 		(pts
+			(xy 161.29 105.41) (xy 152.4 105.41)
+		)
+		(stroke
+			(width 0)
+			(type default)
+		)
+	)
+	(wire
+		(pts
 			(xy 77.47 78.74) (xy 77.47 82.55)
 		)
@@
 	(wire
 		(pts
+			(xy 152.4 118.11) (xy 144.78 118.11)
+		)
+		(stroke
+			(width 0)
+			(type default)
+		)
+	)
+	(wire
+		(pts
+			(xy 152.4 105.41) (xy 152.4 118.11)
+		)
+		(stroke
+			(width 0)
+			(type default)
+		)
+	)
+	(wire
+		(pts
 			(xy 100.33 118.11) (xy 119.38 118.11)
 		)
@@
 	(wire
 		(pts
-			(xy 172.72 118.11) (xy 185.42 118.11)
+			(xy 172.72 118.11) (xy 178.435 118.11)
 		)
 		(stroke
@@
 	(wire
 		(pts
-			(xy 157.48 118.11) (xy 144.78 118.11)
+			(xy 157.48 118.11) (xy 152.4 118.11)
 		)
 		(stroke
@@
 	)
 	(symbol
-		(lib_id "Diode:1N4007")
+		(lib_id "Diode:1N5819")
 		(at 123.19 118.11 180)
 		(unit 1)
@@
 			)
 		)
-		(property "Value" "1N4007"
+		(property "Value" "1N5819"
 			(at 123.19 114.9096 0)
 			(effects
@@
 			)
 		)
-		(property "Datasheet" "http://www.vishay.com/docs/88503/1n4001.pdf"
+		(property "Datasheet" "http://www.vishay.com/docs/88525/1n5817.pdf"
 			(at 123.19 118.11 0)
 			(effects
@@
 			)
 		)
-		(property "Description" ""
+		(property "Description" "40V 1A Schottky Barrier Rectifier Diode, DO-41"
 			(at 123.19 118.11 0)
 			(effects
@@
 					(size 1.27 1.27)
 				)
-			)
-		)
-		(property "LCSC" "C64898"
+				(hide yes)
+			)
+		)
+		(property "LCSC" "C191023"
 			(at 123.19 118.11 0)
 			(effects
@@
 					(unit 1)
 				)
+			)
+		)
+	)
+	(symbol
+		(lib_id "Device:D_Schottky")
+		(at 165.1 105.41 0)
+		(unit 1)
+		(exclude_from_sim no)
+		(in_bom yes)
+		(on_board yes)
+		(dnp no)
+		(property "Reference" "D9"
+			(at 164.7825 99.9955 0)
+			(effects
+				(font
+					(size 1.27 1.27)
+				)
+			)
+		)
+		(property "Value" "1N5819"
+			(at 164.7825 102.4198 0)
+			(effects
+				(font
+					(size 1.27 1.27)
+				)
+			)
+		)
+		(property "Footprint" "Diode_SMD:D_SOD-123"
+			(at 165.1 105.41 0)
+			(effects
+				(font
+					(size 1.27 1.27)
+				)
+				(hide yes)
+			)
+		)
+		(property "Datasheet" "~"
+			(at 165.1 105.41 0)
+			(effects
+				(font
+					(size 1.27 1.27)
+				)
+				(hide yes)
+			)
+		)
+		(property "Description" "Schottky diode"
+			(at 165.1 105.41 0)
+			(effects
+				(font
+					(size 1.27 1.27)
+				)
+				(hide yes)
+			)
+		)
+		(property "LCSC" "C191023"
+			(at 165.1 105.41 0)
+			(effects
+				(font
+					(size 1.27 1.27)
+				)
+				(hide yes)
+			)
+		)
+		(pin "2"
+		)
+		(pin "1"
+		)
+		(instances
+			(project "hwexla"
+				(path "/1cc5480b-56b7-4379-98e2-ccafc88911a7/00000000-0000-0000-0000-000061aa5240"
+					(reference "D9")
+					(unit 1)
+				)
