File: pcb/io.kicad_sch (KiCad schematic)
At the start: 31 parts, among them Q3 2N7002, Q4 2N7002, Q5 2N7002, Q6 2N7002, Q7 BT148, Q8 BT148

Commit message: Fix errors & warnings reported by DRC.
Connections:
- net L-BTN-OUT: now also RN4.6 (R3.2); no longer RN4.7 (R2.2)
- net L-OUT-: now also RN4.7 (R2.2); no longer RN4.6 (R3.2)
- net at RN3.6 (R3.2), RN4.3 (R3.1): now also Q4.1 (G); no longer Q6.1 (G)
- net at RN3.7 (R2.2), RN4.2 (R2.1): now also Q6.1 (G); no longer Q4.1 (G)
Other:
- moved on the sheet: RN3B, RN3C, RN4B, RN4C

Commit message: Use more available resistor grid.
Parts:
- RN4: value 250R -> 470R
Changed lines of the file:
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@@
     (in_bom yes) (on_board yes)
     (property "Reference" "RN4" (id 0) (at 220.98 129.54 90))
-    (property "Value" "250R" (id 1) (at 220.98 132.08 90))
+    (property "Value" "470R" (id 1) (at 220.98 132.08 90))
     (property "Footprint" "Resistor_SMD:R_Array_Concave_4x0603" (id 2) (at 220.98 124.968 90)
       (effects (font (size 1.27 1.27)) hide)
@@
     (in_bom yes) (on_board yes)
     (property "Reference" "RN4" (id 0) (at 220.98 106.68 90))
-    (property "Value" "250R" (id 1) (at 220.98 109.22 90))
+    (property "Value" "470R" (id 1) (at 220.98 109.22 90))
     (property "Footprint" "Resistor_SMD:R_Array_Concave_4x0603" (id 2) (at 220.98 102.108 90)
       (effects (font (size 1.27 1.27)) hide)
@@
     (in_bom yes) (on_board yes)
     (property "Reference" "RN4" (id 0) (at 220.98 144.78 90))
-    (property "Value" "250R" (id 1) (at 220.98 147.32 90))
+    (property "Value" "470R" (id 1) (at 220.98 147.32 90))
     (property "Footprint" "Resistor_SMD:R_Array_Concave_4x0603" (id 2) (at 220.98 140.208 90)
       (effects (font (size 1.27 1.27)) hide)
@@
     (in_bom yes) (on_board yes)
     (property "Reference" "RN4" (id 0) (at 220.98 93.98 90))
-    (property "Value" "250R" (id 1) (at 220.98 91.44 90))
+    (property "Value" "470R" (id 1) (at 220.98 91.44 90))
     (property "Footprint" "Resistor_SMD:R_Array_Concave_4x0603" (id 2) (at 220.98 90.932 90)
       (effects (font (size 1.27 1.27)) hide)

Commit message: Fix bad BT148 pinout & fix connected wires.
Parts:
- Q7, Q8: symbol Triac_Thyristor:BT169D -> Device:Q_SCR_KAG
Connections:
- net GND: now also Q7.1 (K), Q8.1 (K); no longer Q7.3 (K), Q8.3 (K)
- net at C8.1, D18.2 (A), R20.2: now also Q7.3 (G); no longer Q7.2 (G)
- net at C11.1, D14.3, D15.3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: now also Q7.2 (A); no longer Q7.1 (A)
- net at C12.2, D17.3, D19.1 (K): now also Q8.2 (A); no longer Q8.1 (A)
- net at C9.1, D19.2 (A), R21.2: now also Q8.3 (G); no longer Q8.2 (G)
Changed lines of the file:
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@@
     (pin "2")
   )
-  (symbol (lib_id "Triac_Thyristor:BT169D") (at 120.65 163.83 0) (unit 1)
+  (symbol (lib_id "Device:Q_SCR_KAG") (at 120.65 163.83 0) (unit 1)
     (in_bom yes) (on_board yes)
     (property "Reference" "Q7" (id 0) (at 122.8852 162.6616 0)
@@
       (effects (font (size 1.27 1.27)) (justify left))
     )
-    (property "Footprint" "Package_TO_SOT_SMD:SOT-223" (id 2) (at 123.19 165.735 0)
-      (effects (font (size 1.27 1.27) italic) (justify left) hide)
-    )
-    (property "Datasheet" "https://media.digikey.com/pdf/Data%20Sheets/NXP%20PDFs/BT169_Series.pdf" (id 3) (at 120.65 163.83 0)
-      (effects (font (size 1.27 1.27)) (justify left) hide)
+    (property "Footprint" "Package_TO_SOT_SMD:SOT-223" (id 2) (at 120.65 163.83 90)
+      (effects (font (size 1.27 1.27)) hide)
+    )
+    (property "Datasheet" "~" (id 3) (at 120.65 163.83 90)
+      (effects (font (size 1.27 1.27)) hide)
     )
     (property "LCSC" "C256433" (id 4) (at 120.65 163.83 0)
@@
     (pin "2")
   )
-  (symbol (lib_id "Triac_Thyristor:BT169D") (at 158.75 163.83 0) (unit 1)
+  (symbol (lib_id "Device:Q_SCR_KAG") (at 158.75 163.83 0) (unit 1)
     (in_bom yes) (on_board yes)
     (property "Reference" "Q8" (id 0) (at 160.9852 162.6616 0)
@@
       (effects (font (size 1.27 1.27)) (justify left))
     )
-    (property "Footprint" "Package_TO_SOT_SMD:SOT-223" (id 2) (at 161.29 165.735 0)
-      (effects (font (size 1.27 1.27) italic) (justify left) hide)
-    )
-    (property "Datasheet" "https://media.digikey.com/pdf/Data%20Sheets/NXP%20PDFs/BT169_Series.pdf" (id 3) (at 158.75 163.83 0)
-      (effects (font (size 1.27 1.27)) (justify left) hide)
+    (property "Footprint" "Package_TO_SOT_SMD:SOT-223" (id 2) (at 158.75 163.83 90)
+      (effects (font (size 1.27 1.27)) hide)
+    )
+    (property "Datasheet" "~" (id 3) (at 158.75 163.83 90)
+      (effects (font (size 1.27 1.27)) hide)
     )
     (property "LCSC" "C256433" (id 4) (at 158.75 163.83 0)

Commit message: Update libraries, add JLCPCB tooling holes.
Parts:
- D18: footprint Diode_SMD:D_SOT-23_ANK -> Package_TO_SOT_SMD:SOT-23; LCSC (none) -> C962733
- D19: footprint Diode_SMD:D_SOT-23_ANK -> Package_TO_SOT_SMD:SOT-23; LCSC (none) -> C2926248
- RN4: LCSC (none) -> C705088
Connections:
- net at C8.1, Q7.3 (G), R20.2: now also D18.1 (A); no longer D18.2 (A)
- net at C11.1, D14.3, D15.3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: now also D18.3 (K); no longer D18.1 (K)
- net at C12.2, D17.3, Q8.2 (A): now also D19.3 (K); no longer D19.1 (K)
- net at C9.1, Q8.3 (G), R21.2: now also D19.1 (A); no longer D19.2 (A)
Changed lines of the file:
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@@
     (pin "2")
   )
-  (symbol (lib_id "Diode:BZX84Cxx") (at 104.14 163.83 90) (mirror x) (unit 1)
+  (symbol (lib_name "BZX84Cxx_1") (lib_id "Diode:BZX84Cxx") (at 104.14 163.83 90) (mirror x) (unit 1)
     (in_bom yes) (on_board yes)
     (property "Reference" "D18" (id 0) (at 106.172 162.6616 90)
@@
       (effects (font (size 1.27 1.27)) (justify right))
     )
-    (property "Footprint" "Diode_SMD:D_SOT-23_ANK" (id 2) (at 108.585 163.83 0)
+    (property "Footprint" "Package_TO_SOT_SMD:SOT-23" (id 2) (at 108.585 163.83 0)
       (effects (font (size 1.27 1.27)) hide)
     )
@@
       (effects (font (size 1.27 1.27)) hide)
     )
-    (property "LCSC" "" (id 4) (at 104.14 163.83 0)
+    (property "LCSC" "C962733" (id 4) (at 104.14 163.83 0)
       (effects (font (size 1.27 1.27)) hide)
     )
@@
     (pin "1")
     (pin "2")
+    (pin "3")
   )
   (symbol (lib_id "Device:Q_SCR_KAG") (at 120.65 163.83 0) (unit 1)
@@
   (symbol (lib_id "power:GND") (at 104.14 186.69 0) (unit 1)
     (in_bom yes) (on_board yes)
-    (property "Reference" "#PWR044" (id 0) (at 104.14 193.04 0)
+    (property "Reference" "#PWR0124" (id 0) (at 104.14 193.04 0)
       (effects (font (size 1.27 1.27)) hide)
     )
@@
   (symbol (lib_id "power:VCC") (at 116.84 45.72 0) (unit 1)
     (in_bom yes) (on_board yes)
-    (property "Reference" "#PWR036" (id 0) (at 116.84 49.53 0)
+    (property "Reference" "#PWR012" (id 0) (at 116.84 49.53 0)
       (effects (font (size 1.27 1.27)) hide)
     )
@@
   (symbol (lib_id "power:VCC") (at 129.54 45.72 0) (unit 1)
     (in_bom yes) (on_board yes)
-    (property "Reference" "#PWR037" (id 0) (at 129.54 49.53 0)
+    (property "Reference" "#PWR013" (id 0) (at 129.54 49.53 0)
       (effects (font (size 1.27 1.27)) hide)
     )
@@
   (symbol (lib_id "power:VCC") (at 116.84 83.82 0) (unit 1)
     (in_bom yes) (on_board yes)
-    (property "Reference" "#PWR038" (id 0) (at 116.84 87.63 0)
+    (property "Reference" "#PWR014" (id 0) (at 116.84 87.63 0)
       (effects (font (size 1.27 1.27)) hide)
     )
@@
   (symbol (lib_id "power:VCC") (at 129.54 83.82 0) (unit 1)
     (in_bom yes) (on_board yes)
-    (property "Reference" "#PWR039" (id 0) (at 129.54 87.63 0)
+    (property "Reference" "#PWR015" (id 0) (at 129.54 87.63 0)
       (effects (font (size 1.27 1.27)) hide)
     )
@@
       (effects (font (size 1.27 1.27)) (justify right))
     )
-    (property "Footprint" "Diode_SMD:D_SOT-23_ANK" (id 2) (at 146.685 163.83 0)
+    (property "Footprint" "Package_TO_SOT_SMD:SOT-23" (id 2) (at 146.685 163.83 0)
       (effects (font (size 1.27 1.27)) hide)
     )
@@
       (effects (font (size 1.27 1.27)) hide)
     )
-    (property "LCSC" "" (id 4) (at 142.24 163.83 0)
+    (property "LCSC" "C2926248" (id 4) (at 142.24 163.83 0)
       (effects (font (size 1.27 1.27)) hide)
     )
@@
     (pin "1")
     (pin "2")
+    (pin "3")
   )
   (symbol (lib_id "Device:Q_SCR_KAG") (at 158.75 163.83 0) (unit 1)
@@
   (symbol (lib_id "power:GND") (at 142.24 186.69 0) (unit 1)
     (in_bom yes) (on_board yes)
-    (property "Reference" "#PWR045" (id 0) (at 142.24 193.04 0)
+    (property "Reference" "#PWR0123" (id 0) (at 142.24 193.04 0)
       (effects (font (size 1.27 1.27)) hide)
     )
@@
   (symbol (lib_id "power:GND") (at 168.91 134.62 0) (unit 1)
     (in_bom yes) (on_board yes)
-    (property "Reference" "#PWR042" (id 0) (at 168.91 140.97 0)
+    (property "Reference" "#PWR0122" (id 0) (at 168.91 140.97 0)
       (effects (font (size 1.27 1.27)) hide)
     )
@@
   (symbol (lib_id "power:GND") (at 194.31 149.86 0) (unit 1)
     (in_bom yes) (on_board yes)
-    (property "Reference" "#PWR043" (id 0) (at 194.31 156.21 0)
+    (property "Reference" "#PWR0126" (id 0) (at 194.31 156.21 0)
       (effects (font (size 1.27 1.27)) hide)
     )
@@
   (symbol (lib_id "power:GND") (at 168.91 96.52 0) (unit 1)
     (in_bom yes) (on_board yes)
-    (property "Reference" "#PWR040" (id 0) (at 168.91 102.87 0)
+    (property "Reference" "#PWR0121" (id 0) (at 168.91 102.87 0)
       (effects (font (size 1.27 1.27)) hide)
     )
@@
   (symbol (lib_id "power:GND") (at 194.31 111.76 0) (unit 1)
     (in_bom yes) (on_board yes)
-    (property "Reference" "#PWR041" (id 0) (at 194.31 118.11 0)
+    (property "Reference" "#PWR0125" (id 0) (at 194.31 118.11 0)
       (effects (font (size 1.27 1.27)) hide)
     )
@@
       (effects (font (size 1.27 1.27)) hide)
     )
+    (property "LCSC" "C705088" (id 4) (at 220.98 127 0)
+      (effects (font (size 1.27 1.27)) hide)
+    )
     (pin "1")
     (pin "8")
@@
       (effects (font (size 1.27 1.27)) hide)
     )
+    (property "LCSC" "C705088" (id 4) (at 220.98 104.14 0)
+      (effects (font (size 1.27 1.27)) hide)
+    )
     (pin "1")
     (pin "8")
@@
       (effects (font (size 1.27 1.27)) hide)
     )
+    (property "LCSC" "C705088" (id 4) (at 220.98 142.24 0)
+      (effects (font (size 1.27 1.27)) hide)
+    )
     (pin "1")
     (pin "8")
@@
       (effects (font (size 1.27 1.27)) hide)
     )
+    (property "LCSC" "C705088" (id 4) (at 220.98 88.9 0)
+      (effects (font (size 1.27 1.27)) hide)
+    )
     (pin "1")
     (pin "8")
@@
   (symbol (lib_id "power:VCC") (at 115.57 25.4 0) (unit 1)
     (in_bom yes) (on_board yes)
-    (property "Reference" "#PWR035" (id 0) (at 115.57 29.21 0)
-      (effects (font (size 1.27 1.27)) hide)
-    )
+    (property "Reference" "#PWR011" (id 0) (at 115.57 29.21 0)
+      (effects (font (size 1.27 1.27)) hide)
+    )

Commit message: Update LCSC numbers.
Parts:
- F4, F5, F6: LCSC C369153 -> C20797
- RN1, RN3: JLCPCB_CORRECTION (none) -> 0;0;90
Changed lines of the file:
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@@
       (effects (font (size 1.27 1.27)) hide)
     )
-    (property "LCSC" "C369153" (id 4) (at 69.85 58.42 0)
+    (property "LCSC" "C20797" (id 4) (at 69.85 58.42 0)
       (effects (font (size 1.27 1.27)) hide)
     )
@@
       (effects (font (size 1.27 1.27)) hide)
     )
-    (property "LCSC" "C369153" (id 4) (at 69.85 73.66 0)
+    (property "LCSC" "C20797" (id 4) (at 69.85 73.66 0)
       (effects (font (size 1.27 1.27)) hide)
     )
@@
       (effects (font (size 1.27 1.27)) hide)
     )
-    (property "LCSC" "C369153" (id 4) (at 69.85 36.83 0)
+    (property "LCSC" "C20797" (id 4) (at 69.85 36.83 0)
       (effects (font (size 1.27 1.27)) hide)
     )
@@
       (effects (font (size 1.27 1.27)) hide)
     )
+    (property "JLCPCB_CORRECTION" "0;0;90" (id 5) (at 116.84 87.63 0)
+      (effects (font (size 1.27 1.27)) hide)
+    )
     (pin "1")
     (pin "8")
@@
       (effects (font (size 1.27 1.27)) hide)
     )
+    (property "JLCPCB_CORRECTION" "0;0;90" (id 5) (at 116.84 49.53 0)
+      (effects (font (size 1.27 1.27)) hide)
+    )
     (pin "1")
     (pin "8")
@@
       (effects (font (size 1.27 1.27)) hide)
     )
+    (property "JLCPCB_CORRECTION" "0;0;90" (id 5) (at 129.54 49.53 0)
+      (effects (font (size 1.27 1.27)) hide)
+    )
     (pin "1")
     (pin "8")
@@
     )
     (property "LCSC" "C396839" (id 4) (at 129.54 87.63 0)
+      (effects (font (size 1.27 1.27)) hide)
+    )
+    (property "JLCPCB_CORRECTION" "0;0;90" (id 5) (at 129.54 87.63 0)
       (effects (font (size 1.27 1.27)) hide)
     )
@@
       (effects (font (size 1.27 1.27)) hide)
     )
+    (property "JLCPCB_CORRECTION" "0;0;90" (id 5) (at 168.91 92.71 0)
+      (effects (font (size 1.27 1.27)) hide)
+    )
     (pin "1")
     (pin "8")
@@
       (effects (font (size 1.27 1.27)) hide)
     )
+    (property "JLCPCB_CORRECTION" "0;0;90" (id 5) (at 194.31 146.05 0)
+      (effects (font (size 1.27 1.27)) hide)
+    )
     (pin "1")
     (pin "8")
@@
       (effects (font (size 1.27 1.27)) hide)
     )
+    (property "JLCPCB_CORRECTION" "0;0;90" (id 5) (at 194.31 107.95 0)
+      (effects (font (size 1.27 1.27)) hide)
+    )
     (pin "1")
     (pin "8")
@@
       (effects (font (size 1.27 1.27)) hide)
     )
+    (property "JLCPCB_CORRECTION" "0;0;90" (id 5) (at 168.91 130.81 0)
+      (effects (font (size 1.27 1.27)) hide)
+    )
