File: pcb/relay.kicad_sch (KiCad schematic)
At the start: 4 parts, among them K1 HFD2/005, Q2 2N7002

Commit message: Add capacitor to relay power pin.
Parts:
- added C14: (no value), Capacitor_SMD:C_0805_2012Metric, symbol Device:C
Connections:
- net GND: now also C14.2
- net REL-POWER: now also C14.1
Changed lines of the file:
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@@
   (title_block
     (title "hWexla - relay")
+    (date "2022-05-29")
     (company "Model Railroader Club Brno I – KMŽ Brno I – https://kmz-brno.cz/")
     (comment 1 "Jan Horáček")
@@
     (comment 4 "Released under the Creative Commons Attribution-ShareAlike 4.0 License")
   )
+  (junction (at 138.43 109.22) (diameter 0) (color 0 0 0 0)
+  )
   (junction (at 168.91 116.84) (diameter 0) (color 0 0 0 0)
   )
@@
     (stroke (width 0) (type default) (color 0 0 0 0))
   )
-  (wire (pts (xy 144.78 109.22) (xy 138.43 109.22))
+  (wire (pts (xy 138.43 109.22) (xy 144.78 109.22))
     (stroke (width 0) (type default) (color 0 0 0 0))
   )
@@
     (stroke (width 0) (type default) (color 0 0 0 0))
   )
+  (wire (pts (xy 138.43 126.365) (xy 138.43 128.905))
+    (stroke (width 0) (type default) (color 0 0 0 0))
+  )
   (wire (pts (xy 140.97 86.36) (xy 137.16 86.36))
     (stroke (width 0) (type default) (color 0 0 0 0))
@@
   )
   (wire (pts (xy 168.91 120.65) (xy 168.91 116.84))
+    (stroke (width 0) (type default) (color 0 0 0 0))
+  )
+  (wire (pts (xy 138.43 118.745) (xy 138.43 109.22))
     (stroke (width 0) (type default) (color 0 0 0 0))
   )
@@
     (pin "2")
   )
+  (symbol (lib_id "Device:C") (at 138.43 122.555 0) (mirror y) (unit 1)
+    (in_bom yes) (on_board yes)
+    (property "Reference" "C14" (id 0) (at 135.509 121.3866 0)
+      (effects (font (size 1.27 1.27)) (justify left))
+    )
+    (property "Value" "" (id 1) (at 135.509 123.698 0)
+      (effects (font (size 1.27 1.27)) (justify left))
+    )
+    (property "Footprint" "Capacitor_SMD:C_0805_2012Metric" (id 2) (at 137.4648 126.365 0)
+      (effects (font (size 1.27 1.27)) hide)
+    )
+    (property "Datasheet" "~" (id 3) (at 138.43 122.555 0)
+      (effects (font (size 1.27 1.27)) hide)
+    )
+    (property "LCSC" "C45783" (id 4) (at 138.43 122.555 0)
+      (effects (font (size 1.27 1.27)) hide)
+    )
+    (pin "1")
+    (pin "2")
+  )
+  (symbol (lib_id "power:GND") (at 138.43 128.905 0) (mirror y) (unit 1)
+    (in_bom yes) (on_board yes)
+    (property "Reference" "#PWR050" (id 0) (at 138.43 135.255 0)
+      (effects (font (size 1.27 1.27)) hide)
+    )
+    (property "Value" "GND" (id 1) (at 138.303 133.2992 0))
+    (property "Footprint" "" (id 2) (at 138.43 128.905 0)
+      (effects (font (size 1.27 1.27)) hide)
+    )
+    (property "Datasheet" "" (id 3) (at 138.43 128.905 0)
+      (effects (font (size 1.27 1.27)) hide)
+    )
+    (pin "1")
+  )
 )

Commit message: Fix relay footprint.
Parts:
- C14: value (none) -> 22u
Connections:
- net RELA+: now also K1.10; no longer K1.8
- net RELA-: now also K1.8; no longer K1.10
- net RELB+: now also K1.3; no longer K1.5
- net RELB-: now also K1.5; no longer K1.3
Changed lines of the file:
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@@
     (stroke (width 0) (type default) (color 0 0 0 0))
   )
-  (wire (pts (xy 140.97 81.28) (xy 137.16 81.28))
+  (wire (pts (xy 140.97 76.2) (xy 137.16 76.2))
     (stroke (width 0) (type default) (color 0 0 0 0))
   )
@@
     (stroke (width 0) (type default) (color 0 0 0 0))
   )
-  (wire (pts (xy 140.97 86.36) (xy 137.16 86.36))
+  (wire (pts (xy 140.97 91.44) (xy 137.16 91.44))
     (stroke (width 0) (type default) (color 0 0 0 0))
   )
@@
     (stroke (width 0) (type default) (color 0 0 0 0))
   )
-  (wire (pts (xy 140.97 76.2) (xy 137.16 76.2))
+  (wire (pts (xy 140.97 81.28) (xy 137.16 81.28))
     (stroke (width 0) (type default) (color 0 0 0 0))
   )
@@
     (stroke (width 0) (type default) (color 0 0 0 0))
   )
-  (wire (pts (xy 140.97 91.44) (xy 137.16 91.44))
+  (wire (pts (xy 140.97 86.36) (xy 137.16 86.36))
     (stroke (width 0) (type default) (color 0 0 0 0))
   )
@@
     (effects (font (size 1.27 1.27)) (justify right))
   )
-  (hierarchical_label "RELA-" (shape bidirectional) (at 137.16 81.28 180)
+  (hierarchical_label "RELA-" (shape bidirectional) (at 137.16 76.2 180)
     (effects (font (size 1.27 1.27)) (justify right))
   )
-  (hierarchical_label "RELA+" (shape bidirectional) (at 137.16 76.2 180)
+  (hierarchical_label "RELA+" (shape bidirectional) (at 137.16 81.28 180)
     (effects (font (size 1.27 1.27)) (justify right))
   )
@@
     (effects (font (size 1.27 1.27)) (justify left))
   )
-  (hierarchical_label "RELB+" (shape bidirectional) (at 137.16 86.36 180)
+  (hierarchical_label "RELB+" (shape bidirectional) (at 137.16 91.44 180)
     (effects (font (size 1.27 1.27)) (justify right))
   )
-  (hierarchical_label "RELB-" (shape bidirectional) (at 137.16 91.44 180)
+  (hierarchical_label "RELB-" (shape bidirectional) (at 137.16 86.36 180)
     (effects (font (size 1.27 1.27)) (justify right))
   )
@@
       (effects (font (size 1.27 1.27)) (justify left))
     )
-    (property "Value" "" (id 1) (at 135.509 123.698 0)
+    (property "Value" "22u" (id 1) (at 135.509 123.698 0)
       (effects (font (size 1.27 1.27)) (justify left))
     )

Commit message: Change relay part.
Parts:
- K1: value HFD2/005 -> RS-5
Changed lines of the file:
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@@
     (in_bom yes) (on_board yes)
     (property "Reference" "K1" (id 0) (at 148.59 69.4182 90))
-    (property "Value" "HFD2/005" (id 1) (at 148.59 71.7296 90))
+    (property "Value" "RS-5" (id 1) (at 148.59 71.7296 90))
     (property "Footprint" "hwexla:HFD2" (id 2) (at 148.59 88.9 0)
       (effects (font (size 1.27 1.27)) hide)

Commit message: Add possible fuses to relays.
Parts:
- added F11, F12: 2A, Fuse:Fuse_1206_3216Metric_Pad1.42x1.75mm_HandSolder, symbol Device:Fuse
Connections:
- net RELA0: now also F11.2; no longer K1.9
- net RELB0: now also F12.2; no longer K1.4
- new net: F12.1, K1.4
- new net: F11.1, K1.9
Other:
- note added: "Do not fit fuses"
Changed lines of the file:
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@@
     (stroke (width 0) (type default) (color 0 0 0 0))
   )
-  (wire (pts (xy 156.21 88.9) (xy 160.02 88.9))
+  (wire (pts (xy 168.275 88.9) (xy 177.165 88.9))
     (stroke (width 0) (type default) (color 0 0 0 0))
   )
@@
     (stroke (width 0) (type default) (color 0 0 0 0))
   )
+  (wire (pts (xy 156.21 88.9) (xy 160.655 88.9))
+    (stroke (width 0) (type default) (color 0 0 0 0))
+  )
   (wire (pts (xy 181.61 109.22) (xy 194.31 109.22))
     (stroke (width 0) (type default) (color 0 0 0 0))
@@
     (stroke (width 0) (type default) (color 0 0 0 0))
   )
+  (wire (pts (xy 156.21 78.74) (xy 160.655 78.74))
+    (stroke (width 0) (type default) (color 0 0 0 0))
+  )
   (wire (pts (xy 140.97 86.36) (xy 137.16 86.36))
     (stroke (width 0) (type default) (color 0 0 0 0))
   )
-  (wire (pts (xy 156.21 78.74) (xy 160.02 78.74))
+  (wire (pts (xy 168.275 78.74) (xy 177.165 78.74))
     (stroke (width 0) (type default) (color 0 0 0 0))
   )
@@
     (stroke (width 0) (type default) (color 0 0 0 0))
   )
-  (hierarchical_label "RELA0" (shape bidirectional) (at 160.02 78.74 0)
+  (text "Do not fit fuses" (at 161.29 74.295 0)
+    (effects (font (size 1.27 1.27)) (justify left bottom))
+  )
+  (hierarchical_label "RELA0" (shape bidirectional) (at 177.165 78.74 0)
     (effects (font (size 1.27 1.27)) (justify left))
   )
@@
     (effects (font (size 1.27 1.27)) (justify right))
   )
-  (hierarchical_label "RELB0" (shape bidirectional) (at 160.02 88.9 0)
+  (hierarchical_label "RELB0" (shape bidirectional) (at 177.165 88.9 0)
     (effects (font (size 1.27 1.27)) (justify left))
   )
@@
       (effects (font (size 1.27 1.27)) hide)
     )
+    (pin "1")
+    (pin "2")
+  )
+  (symbol (lib_id "Device:Fuse") (at 164.465 78.74 90) (unit 1)
+    (in_bom yes) (on_board yes)
+    (property "Reference" "F11" (id 0) (at 164.465 80.645 90))
+    (property "Value" "2A" (id 1) (at 164.465 76.8151 90))
+    (property "Footprint" "Fuse:Fuse_1206_3216Metric_Pad1.42x1.75mm_HandSolder" (id 2) (at 164.465 80.518 90)
+      (effects (font (size 1.27 1.27)) hide)
+    )
+    (property "Datasheet" "~" (id 3) (at 164.465 78.74 0)
+      (effects (font (size 1.27 1.27)) hide)
+    )
+    (property "LCSC" "C17477" (id 4) (at 164.465 78.74 90)
+      (effects (font (size 1.27 1.27)) hide)
+    )
+    (pin "1")
+    (pin "2")
+  )
+  (symbol (lib_id "Device:Fuse") (at 164.465 88.9 90) (unit 1)
+    (in_bom yes) (on_board yes)
+    (property "Reference" "F12" (id 0) (at 164.465 90.805 90))
+    (property "Value" "2A" (id 1) (at 164.465 86.9751 90))
+    (property "Footprint" "Fuse:Fuse_1206_3216Metric_Pad1.42x1.75mm_HandSolder" (id 2) (at 164.465 90.678 90)
+      (effects (font (size 1.27 1.27)) hide)
+    )
+    (property "Datasheet" "~" (id 3) (at 164.465 88.9 0)
+      (effects (font (size 1.27 1.27)) hide)
+    )
+    (property "LCSC" "C17477" (id 4) (at 164.465 88.9 90)
+      (effects (font (size 1.27 1.27)) hide)
+    )

Commit message: Update libraries, add JLCPCB tooling holes.
Parts:
- K1: JLCPCB_IGNORE (none) -> true
Changed lines of the file:
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@@
+      (effects (font (size 1.27 1.27)) hide)
+    )
+    (property "JLCPCB_IGNORE" "true" (id 4) (at 148.59 88.9 0)
       (effects (font (size 1.27 1.27)) hide)
     )
@@
   (symbol (lib_id "power:GND") (at 168.91 120.65 0) (unit 1)
     (in_bom yes) (on_board yes)
-    (property "Reference" "#PWR034" (id 0) (at 168.91 127 0)
+    (property "Reference" "#PWR0134" (id 0) (at 168.91 127 0)
       (effects (font (size 1.27 1.27)) hide)
     )
@@
   (symbol (lib_id "power:GND") (at 138.43 128.905 0) (mirror y) (unit 1)
     (in_bom yes) (on_board yes)
-    (property "Reference" "#PWR050" (id 0) (at 138.43 135.255 0)
+    (property "Reference" "#PWR0133" (id 0) (at 138.43 135.255 0)
       (effects (font (size 1.27 1.27)) hide)
     )

Commit message: Update LCSC numbers.
Parts:
- F11, F12: LCSC C17477 -> C17888
Changed lines of the file:
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@@
       (effects (font (size 1.27 1.27)) hide)
     )
-    (property "LCSC" "C17477" (id 4) (at 164.465 78.74 90)
+    (property "LCSC" "C17888" (id 4) (at 164.465 78.74 90)
       (effects (font (size 1.27 1.27)) hide)
     )
@@
       (effects (font (size 1.27 1.27)) hide)
     )
-    (property "LCSC" "C17477" (id 4) (at 164.465 88.9 90)
+    (property "LCSC" "C17888" (id 4) (at 164.465 88.9 90)
       (effects (font (size 1.27 1.27)) hide)
     )
