File: pcb/relay.kicad_sch (KiCad schematic)
At the start: 7 parts, among them K1 RS-5, Q2 2N7002

Commit message: Add protection on internal inputs, divide stepdown voltage measuring by 2.
Parts:
- added R14: 1k, Resistor_SMD:R_0805_2012Metric_Pad1.20x1.40mm_HandSolder, symbol Device:R
Connections:
- net REL-CONTROL: now also R14.2; no longer Q2.1 (G), R11.1
- new net: Q2.1 (G), R11.1, R14.1
Other:
- moved on the sheet: C14, D13, F11, F12, K1, Q2, R11
