File: pcb/relay.kicad_sch (KiCad schematic)
At the start: 8 parts, among them K1 RS-5, Q2 2N7002

Commit message: REL: fix bad wire names.
Connections:
- net RELA+: now also K1.8; no longer K1.10
- net RELA-: now also K1.10; no longer K1.8
- net RELB+: now also K1.5; no longer K1.3
- net RELB-: now also K1.3; no longer K1.5
Changed lines of the file:
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@@
 		)
 	)
-	(hierarchical_label "RELA-"
+	(hierarchical_label "RELA+"
 		(shape bidirectional)
 		(at 119.38 77.47 180)
@@
 		)
 	)
-	(hierarchical_label "RELA+"
+	(hierarchical_label "RELA-"
 		(shape bidirectional)
 		(at 119.38 82.55 180)
@@
 		)
 	)
-	(hierarchical_label "RELB+"
+	(hierarchical_label "RELB-"
 		(shape bidirectional)
 		(at 119.38 92.71 180)
@@
 		)
 	)
-	(hierarchical_label "RELB-"
+	(hierarchical_label "RELB+"
 		(shape bidirectional)
 		(at 119.38 87.63 180)
