File: diagpcb/hwexladiag.kicad_pcb (KiCad board)
At the start: 2 copper layers, 20 x 30 mm, 17 parts, among them J1 PINHEADER, Q1 2N7002, Q2 2N7002, SW1 SW_Push, U1 HC05, U2 HT75xx-1-SOT89

Commit message: diag: remove blue LED.
Parts:
- removed D2: BLUE, LED_SMD:LED_0805_2012Metric
- removed R6: 1k, Resistor_SMD:R_0805_2012Metric
- U2: value HT75xx-1-SOT89 -> HT7533-1
Routing:
- net Net-(U1-PIO11): track 41.3 -> 38.3 mm
- net Net-(D2-A): track 2.30 -> 0.00 mm
- net GND: vias 16 -> 15

Commit message: diag: pin 31 for red LED.
Connections:
- R5 pad 1: Net-(U1-PIO10) -> Net-(U1-PIO8)
- U1 pad 31: unconnected-(U1-PIO8-Pad31) -> Net-(U1-PIO8)
- U1 pad 33: Net-(U1-PIO10) -> unconnected-(U1-PIO10-Pad33)
Routing:
- net Net-(U1-PIO10): track 31.0 -> 0.00 mm, vias 2 -> 0
- net Net-(U1-PIO8): track 0.00 -> 29.8 mm, vias 0 -> 2

Commit message: diag: use input resistor 10R.
Parts:
- added R6: 10R, Resistor_SMD:R_0805_2012Metric, B.Cu at (148.3, 92.7)
Connections:
- C1 pad 1: +5V -> Net-(U2-VIN)
- U2 pad 2: +5V -> Net-(U2-VIN)
Routing:
- net Net-(U2-VIN): track 0.00 -> 4.73 mm
- net +5V: track 26.3 -> 24.0 mm
- net Net-(U1-PIO11): track 38.3 -> 39.6 mm
- net Net-(U1-PIO8): track 29.8 -> 28.7 mm
- net +3V3: track 49.0 -> 49.6 mm

Commit message: Use smaller HC05 footprint.
Make the PCB smaller by 2.8 mm.
Parts:
- moved C2 1.84 mm to (153.6, 91.6), turned to 90 degrees
- moved U2 1.81 mm to (152.4, 96.2)
- moved D1 1.34 mm to (153.6, 82.5)
- moved R5 1.34 mm to (151.3, 82.5)
- moved J1 1.21 mm to (142.4, 89.1)
- moved SW1 1.21 mm to (142.9, 82.7)
- moved C1 1.11 mm to (148.3, 96.5)
- moved Q1 0.76 mm to (149.5, 103.3)
- moved Q2 0.76 mm to (145.0, 103.3)
- moved R1 0.76 mm to (149.5, 100.0)
- moved R2 0.76 mm to (149.5, 106.6)
- moved R3 0.76 mm to (145.0, 100.0)
- moved R4 0.76 mm to (145.0, 106.6)
- moved R7 0.26 mm to (150.6, 82.5)
- moved R6 0.20 mm to (148.5, 92.6)
Routing:
- net +3V3: track 49.6 -> 53.6 mm
- net Net-(U1-PIO11): track 39.6 -> 37.5 mm
- net Net-(U2-VIN): track 4.73 -> 5.92 mm
- net Net-(U1-PIO8): track 28.7 -> 27.6 mm
- net /HCTX: track 14.3 -> 13.5 mm
- net /HCRX: track 9.88 -> 9.14 mm
- net /wexlaRxD: track 15.5 -> 16.2 mm
- net +5V: track 24.0 -> 23.5 mm
- net GND: track 2.57 -> 2.32 mm, vias 15 -> 14
Other:
- board size 20 x 30 mm -> 17.2 x 30 mm
- board text added: "JH 2024 v1.1"
- board text removed: "JH 2023 v1.0"

Commit message: Add jumper for AT pin external connection.
Parts:
- added JP1: ~, Jumper:SolderJumper-2_P1.3mm_Open_RoundedPad1.0x1.5mm, B.Cu at (148.5, 82.7)
- R5: value 1k -> 4k7
- moved R7 2.30 mm to (152.8, 82.7)
Connections:
- J1 pad 1: unconnected-(J1-Pin_1-Pad1) -> AT
Routing:
- net AT: track 0.00 -> 3.79 mm
- net Net-(JP1-A): track 37.5 -> 39.9 mm
- net GND: vias 14 -> 16
- net +5V: vias 3 -> 2
Other:
- board text added: "AT"
- board text added: "AT RX TX +5V NC GND"
- board text added: "RX"
- board text added: "TX"
