File: wexlacon/wexlacon.kicad_pcb (KiCad board)
At the start: 2 copper layers, 42 x 50 mm, 15 parts, among them J1 CAN25, J2 MVE252-5-V, J3 solder, J4 MVE253-5-V, J5 KK-254, J9 pinheader

Commit message: Enlarge CAN screwdriver holes.
Other:
- outline, holes or cut-outs redrawn
Changed lines of the file:
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@@
 	)
 	(gr_line
-		(start 151.6 130)
+		(start 152.6 130)
 		(end 170 130)
 		(stroke
@@
 		(layer "Edge.Cuts")
 	)
+	(gr_arc
+		(start 151.199999 81.400001)
+		(mid 150.614213 82.814215)
+		(end 149.199999 83.400001)
+		(stroke
+			(width 0.05)
+			(type default)
+		)
+		(layer "Edge.Cuts")
+	)
+	(gr_arc
+		(start 143.799999 80.000001)
+		(mid 144.789948 80.410052)
+		(end 145.199999 81.400001)
+		(stroke
+			(width 0.05)
+			(type default)
+		)
+		(layer "Edge.Cuts")
+	)
 	(gr_line
 		(start 132 80)
-		(end 144.8 80)
+		(end 143.8 80)
 		(stroke
 			(width 0.05)
@@
 	)
 	(gr_line
-		(start 144.8 130)
+		(start 143.8 130)
 		(end 132 130)
 		(stroke
@@
 	)
 	(gr_arc
-		(start 146.2 128.6)
-		(mid 145.789949 129.589949)
-		(end 144.8 130)
+		(start 151.199999 81.400001)
+		(mid 151.61005 80.410052)
+		(end 152.599999 80.000001)
 		(stroke
 			(width 0.05)
@@
 	)
 	(gr_arc
-		(start 150.2 81.4)
-		(mid 150.610051 80.410051)
-		(end 151.6 80)
+		(start 145.2 128.6)
+		(mid 145.785786 127.185786)
+		(end 147.2 126.6)
 		(stroke
 			(width 0.05)
@@
 	)
 	(gr_arc
-		(start 150.2 81.4)
-		(mid 148.2 83.4)
-		(end 146.2 81.4)
+		(start 145.2 128.6)
+		(mid 144.789949 129.589949)
+		(end 143.8 130)
 		(stroke
 			(width 0.05)
@@
 	)
 	(gr_arc
-		(start 151.6 130)
-		(mid 150.610051 129.589949)
-		(end 150.2 128.6)
+		(start 147.2 83.4)
+		(mid 145.785786 82.814214)
+		(end 145.2 81.4)
+		(stroke
+			(width 0.05)
+			(type default)
+		)
+		(layer "Edge.Cuts")
+	)
+	(gr_line
+		(start 149.199999 126.600001)
+		(end 147.2 126.600001)
+		(stroke
+			(width 0.05)
+			(type default)
+		)
+		(layer "Edge.Cuts")
+	)
+	(gr_arc
+		(start 149.199999 126.600001)
+		(mid 150.614213 127.185787)
+		(end 151.199999 128.600001)
+		(stroke
+			(width 0.05)
+			(type default)
+		)
+		(layer "Edge.Cuts")
+	)
+	(gr_arc
+		(start 152.6 130)
+		(mid 151.610051 129.589949)
+		(end 151.2 128.6)
 		(stroke
 			(width 0.05)
@@
 	)
 	(gr_line
-		(start 130 128)
-		(end 130 82)
+		(start 147.2 83.4)
+		(end 149.199999 83.4)
 		(stroke
 			(width 0.05)
@@
 		(layer "Edge.Cuts")
 	)
-	(gr_arc
-		(start 146.2 128.6)
-		(mid 148.2 126.6)
-		(end 150.2 128.6)
+	(gr_line
+		(start 130 128)
+		(end 130 82)
 		(stroke
 			(width 0.05)
@@
 		(layer "Edge.Cuts")
 	)
-	(gr_arc
-		(start 144.8 80)
-		(mid 145.789949 80.410051)
-		(end 146.2 81.4)
+	(gr_line
+		(start 170 80)
+		(end 152.6 80)
 		(stroke
 			(width 0.05)
-			(type default)
-		)
-		(layer "Edge.Cuts")
-	)
-	(gr_line
-		(start 170 80)
-		(end 151.6 80)
-		(stroke
-			(width 0.05)

Commit message: Several minor enahncements.
* Corners: larger diameter (smaller PCB).
* Mark turnout wire hole on silkscreen.
* Unify connector names with WexlaCon v3.
* Use D-SUB25 schematic symbol without holes.
Parts:
- removed J4: MVE253-5-V, relaycon:RELAYCON
- removed the J5 at (133.6, 102.8)
- added J10: solder, relaycon:RELAYCON, F.Cu at (159.2, 91.6)
- added J6: pinheader, Connector_PinHeader_2.54mm:PinHeader_2x04_P2.54mm_Vertical, F.Cu at (161.0, 127.0)
- J3: value solder -> KK-254; footprint relaycon:RELAYCON -> Connector_Molex:Molex_KK-254_AE-6410-04A_1x04_P2.54mm_Vertical
- J9: value pinheader -> MVE253-5-V; footprint Connector_PinHeader_2.54mm:PinHeader_2x04_P2.54mm_Vertical -> relaycon:RELAYCON
- moved J9 35.8 mm to (166.8, 91.6)
- moved J3 28.0 mm to (133.6, 102.8)
- renumbered J2 to J1, J1 to J5
Connections:
- J3 pad 1: RELB- -> BTN+
- J3 pad 2: RELB0 -> BTN-
- J3 pad 3: RELB+ -> GND
- J9 pad 1: GND -> RELA+
- J9 pad 2: IN-SLAVE -> RELA0
- J9 pad 3: IN- -> RELA-
Other:
- outline, holes or cut-outs redrawn

Commit message: Adapter drill d=1.8 mm.
Parts:
- removed H4, H6: 1.0mm, TestPoint:TestPoint_THTPad_D2.0mm_Drill1.0mm
Routing:
- net (no net): vias 0 -> 2
Changed lines of the file:
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@@
-		)
-	)
-	(footprint "TestPoint:TestPoint_THTPad_D2.0mm_Drill1.0mm"
-		(layer "F.Cu")
-		(at 161.3 103.5)
-		(descr "THT pad as test Point, diameter 2.0mm, hole diameter 1.0mm")
-		(tags "test point THT pad")
-		(property "Reference" "H4"
-			(at 0 -1.998 0)
-			(layer "F.SilkS")
-			(hide yes)
-			(effects
-				(font
-					(size 1 1)
-					(thickness 0.15)
-				)
-			)
-		)
-		(property "Value" "1.0mm"
-			(at 0 2.05 0)
-			(layer "F.Fab")
-			(effects
-				(font
-					(size 1 1)
-					(thickness 0.15)
-				)
-			)
-		)
-		(property "Footprint" "TestPoint:TestPoint_THTPad_D2.0mm_Drill1.0mm"
-			(at 0 0 0)
-			(unlocked yes)
-			(layer "F.Fab")
-			(hide yes)
-			(effects
-				(font
-					(size 1.27 1.27)
-					(thickness 0.15)
-				)
-			)
-		)
-		(property "Datasheet" ""
-			(at 0 0 0)
-			(unlocked yes)
-			(layer "F.Fab")
-			(hide yes)
-			(effects
-				(font
-					(size 1.27 1.27)
-					(thickness 0.15)
-				)
-			)
-		)
-		(property "Description" "Mounting Hole without connection"
-			(at 0 0 0)
-			(unlocked yes)
-			(layer "F.Fab")
-			(hide yes)
-			(effects
-				(font
-					(size 1.27 1.27)
-					(thickness 0.15)
-				)
-			)
-		)
-		(property ki_fp_filters "MountingHole*")
-		(sheetname "Root")
-		(sheetfile "wexlacon.kicad_sch")
-		(attr exclude_from_pos_files exclude_from_bom)
-		(fp_circle
-			(center 0 0)
-			(end 0 1.2)
-			(stroke
-				(width 0.12)
-				(type solid)
-			)
-			(fill none)
-			(layer "F.SilkS")
-		)
-		(fp_circle
-			(center 0 0)
-			(end 1.5 0)
-			(stroke
-				(width 0.05)
-				(type solid)
-			)
-			(fill none)
-			(layer "F.CrtYd")
-		)
-		(fp_text user "${REFERENCE}"
-			(at 0 -2 0)
-			(layer "F.Fab")
-			(effects
-				(font
-					(size 1 1)
-					(thickness 0.15)
-				)
-			)
-		)
-		(pad "1" thru_hole circle
-			(at 0 0)
-			(size 2 2)
-			(drill 1)
-			(layers "*.Cu" "*.Mask")
-			(remove_unused_layers no)
 		)
 	)
@@
 		)
 	)
-	(footprint "TestPoint:TestPoint_THTPad_D2.0mm_Drill1.0mm"
-		(layer "F.Cu")
-		(at 161.3 115.5)
-		(descr "THT pad as test Point, diameter 2.0mm, hole diameter 1.0mm")
-		(tags "test point THT pad")
-		(property "Reference" "H6"
-			(at 0 -1.998 0)
-			(layer "F.SilkS")
-			(hide yes)
-			(effects
-				(font
-					(size 1 1)
-					(thickness 0.15)
-				)
-			)
-		)
-		(property "Value" "1.0mm"
-			(at 0 2.05 0)
-			(layer "F.Fab")
-			(effects
-				(font
-					(size 1 1)
-					(thickness 0.15)
-				)
-			)
-		)
-		(property "Footprint" "TestPoint:TestPoint_THTPad_D2.0mm_Drill1.0mm"
-			(at 0 0 0)
-			(unlocked yes)
-			(layer "F.Fab")
-			(hide yes)
-			(effects
-				(font
-					(size 1.27 1.27)
-					(thickness 0.15)
-				)
-			)
-		)
-		(property "Datasheet" ""
-			(at 0 0 0)
-			(unlocked yes)
-			(layer "F.Fab")
-			(hide yes)
-			(effects
-				(font
-					(size 1.27 1.27)
-					(thickness 0.15)
-				)
-			)
-		)
-		(property "Description" "Mounting Hole without connection"
-			(at 0 0 0)
-			(unlocked yes)
-			(layer "F.Fab")
-			(hide yes)
-			(effects
-				(font
-					(size 1.27 1.27)
-					(thickness 0.15)
-				)
-			)
-		)
-		(property ki_fp_filters "MountingHole*")
-		(sheetname "Root")
-		(sheetfile "wexlacon.kicad_sch")
-		(attr exclude_from_pos_files exclude_from_bom)
-		(fp_circle
-			(center 0 0)
-			(end 0 1.2)
-			(stroke
-				(width 0.12)
-				(type solid)
-			)
-			(fill none)
-			(layer "F.SilkS")
-		)
-		(fp_circle
-			(center 0 0)
-			(end 1.5 0)
-			(stroke
-				(width 0.05)
-				(type solid)
-			)
-			(fill none)
-			(layer "F.CrtYd")
-		)
-		(fp_text user "${REFERENCE}"
-			(at 0 -2 0)
-			(layer "F.Fab")
-			(effects
-				(font
-					(size 1 1)
-					(thickness 0.15)
-				)
-			)
-		)
-		(pad "1" thru_hole circle
-			(at 0 0)
-			(size 2 2)
-			(drill 1)
-			(layers "*.Cu" "*.Mask")
-			(remove_unused_layers no)
-		)
-	)
 	(footprint "MountingHole:MountingHole_3.2mm_M3_Pad"
 		(layer "F.Cu")
@@
 		)
 	)
+	(via
+		(at 161.3 103.5)
+		(size 2.5)
+		(drill 1.8)
+		(layers "F.Cu" "B.Cu")
+		(net 0)
+	)
+	(via
+		(at 161.3 115.5)
+		(size 2.5)
+		(drill 1.8)
+		(layers "F.Cu" "B.Cu")
+		(net 0)
+	)
 	(segment

Commit message: Fix switched order of relay contacts.
Connections:
- J10 pad 1: RELB- -> RELB+
- J10 pad 3: RELB+ -> RELB-
- J5 pad 12: RELB+ -> RELB-
- J5 pad 13: RELB+ -> RELB-
- J5 pad 20: RELA+ -> RELA-
- J5 pad 21: RELA+ -> RELA-
- J5 pad 24: RELA- -> RELA+
- J5 pad 25: RELA- -> RELA+
- J5 pad 8: RELB- -> RELB+
- J5 pad 9: RELB- -> RELB+
- J9 pad 1: RELA+ -> RELA-
- J9 pad 3: RELA- -> RELA+
Routing:
- net RELA-: track 30.2 -> 65.3 mm
- net RELA+: track 65.3 -> 30.2 mm
Other:
- board text added: "JM 2026"
- board text added: "WEXLACON v4.1"
- board text added: "rel. A -0+"
- board text added: "rel. B +0-"
- board text removed: "JH 2025"
- board text removed: "WEXLACON v4.0"
- board text removed: "rel. A +0-"
- board text removed: "rel. B -0+"
