File: wexlacon/wexlacon.kicad_sch (KiCad schematic)
At the start: 18 parts, among them J1 CAN25, J2 Screw_Terminal_01x02, J3 Screw_Terminal_01x03, J4 Screw_Terminal_01x03, J5 Conn_01x04, J6 Conn_01x02, J7 Conn_01x02, J8 Conn_01x02

Commit message: wexlacon: pcb.
Parts:
- removed J6, J7, J8: Conn_01x02, symbol Connector_Generic:Conn_01x02
- removed JP1: pinheader, Connector_PinHeader_2.54mm:PinHeader_1x02_P2.54mm_Vertical, symbol Jumper:Jumper_2_Open
- added J9: pinheader, Connector_PinHeader_2.54mm:PinHeader_2x04_P2.54mm_Vertical, symbol Connector_Generic:Conn_02x04_Odd_Even
- H4, H5, H6: value ~ -> 1.0mm; footprint (none) -> TestPoint:TestPoint_THTPad_D2.0mm_Drill1.0mm
- J1: footprint Connector_Dsub:DSUB-25_Female_Vertical_P2.77x2.84mm_MountingHoles -> Connector_Dsub:DSUB-25_Female_Vertical_P2.77x2.84mm
- J2: value Screw_Terminal_01x02 -> MVE252-5-V; footprint (none) -> TerminalBlock_Euroclamp:MVE252-5-V
- J3: value Screw_Terminal_01x03 -> solder; footprint (none) -> relaycon:RELAYCON; symbol Connector:Screw_Terminal_01x03 -> Connector_Generic:Conn_01x03
- J4: value Screw_Terminal_01x03 -> MVE253-5-V; footprint (none) -> relaycon:RELAYCON
- J5: value Conn_01x04 -> KK-254
- R1: renamed from R3; footprint Resistor_SMD:R_1206_3216Metric -> Resistor_SMD:R_1206_3216Metric_Pad1.30x1.75mm_HandSolder
- R2: footprint Resistor_SMD:R_1206_3216Metric -> Resistor_SMD:R_1206_3216Metric_Pad1.30x1.75mm_HandSolder
- R3: renamed from R1; footprint Resistor_SMD:R_1206_3216Metric -> Resistor_SMD:R_1206_3216Metric_Pad1.30x1.75mm_HandSolder
Connections:
- net BTN+: now also J9.7 (Pin_7)
- net BTN-: now also J9.8 (Pin_8)
- net GND: now also J9.1 (Pin_1)
- net IN+: now also J9.4 (Pin_4)
- net IN-: now also J9.3 (Pin_3)
- net IN-SLAVE: now also J9.2 (Pin_2)
- net OUT+: now also J9.5 (Pin_5)
- net OUT-: now also J9.6 (Pin_6)
- net RELAL renamed RELB-
- net RELAM renamed RELB0
- net RELAR renamed RELB+
- net RELBL renamed RELA-
- net RELA-: now also J4.3 (Pin_3); no longer J4.1 (Pin_1)
- net RELBM renamed RELA0
- net RELBR renamed RELA+
- net RELA+: now also J4.1 (Pin_1); no longer J4.3 (Pin_3)
Other:
- moved on the sheet: J4, J5, R1, R2, R3

Commit message: Enlarge CAN screwdriver holes.
Other:
- note added: "Mounting holes"
- note added: "Turnout wire holes"
Changed lines of the file:
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@@
+		)
+	)
+	(text "Mounting holes"
+		(exclude_from_sim no)
+		(at 39.37 113.03 0)
+		(effects
+			(font
+				(size 1.27 1.27)
+			)
+		)
+	)
+	(text "Turnout wire\nholes"
+		(exclude_from_sim no)
+		(at 69.85 111.76 0)
+		(effects
+			(font
+				(size 1.27 1.27)
+			)
 		)
 	)

Commit message: Several minor enahncements.
* Corners: larger diameter (smaller PCB).
* Mark turnout wire hole on silkscreen.
* Unify connector names with WexlaCon v3.
* Use D-SUB25 schematic symbol without holes.
Parts:
- J5: renamed from J1; symbol Connector:DB25_Receptacle_MountingHoles -> Connector:DB25_Receptacle
- renumbered J2 to J1, J3 to J10, J5 to J3, J9 to J6, J4 to J9
Connections:
- no-connect marks 2 -> 1
Changed lines of the file:
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@@
 		(at 173.99 48.26)
 	)
-	(no_connect
-		(at 181.61 91.44)
-	)
 	(wire
 		(pts
@@
 		(on_board yes)
 		(dnp no)
-		(property "Reference" "J9"
+		(property "Reference" "J6"
 			(at 97.79 30.1455 0)
 			(effects
@@
 			(project ""
 				(path "/0fece1c8-c6d0-4b5d-a04d-4f9ff43ff97c"
-					(reference "J9")
+					(reference "J6")
 					(unit 1)
 				)
@@
 	)
 	(symbol
-		(lib_id "Connector:DB25_Receptacle_MountingHoles")
+		(lib_id "Connector:DB25_Receptacle")
 		(at 181.61 55.88 0)
 		(unit 1)
@@
 		(on_board yes)
 		(dnp no)
-		(property "Reference" "J1"
+		(property "Reference" "J5"
 			(at 186.182 54.6678 0)
 			(effects
@@
 			)
 		)
-		(property "Description" "25-pin female receptacle socket D-SUB connector, Mounting Hole"
+		(property "Description" "25-pin female receptacle socket D-SUB connector"
 			(at 181.61 55.88 0)
 			(effects
@@
 		(pin "25"
 		)
-		(pin "0"
-		)
 		(pin "20"
 		)
@@
 			(project ""
 				(path "/0fece1c8-c6d0-4b5d-a04d-4f9ff43ff97c"
-					(reference "J1")
+					(reference "J5")
 					(unit 1)
 				)
@@
 		(dnp no)
 		(fields_autoplaced yes)
-		(property "Reference" "J5"
+		(property "Reference" "J3"
 			(at 26.67 42.8455 0)
 			(effects
@@
 			(project ""
 				(path "/0fece1c8-c6d0-4b5d-a04d-4f9ff43ff97c"
-					(reference "J5")
+					(reference "J3")
 					(unit 1)
 				)
@@
 		(dnp no)
 		(fields_autoplaced yes)
-		(property "Reference" "J4"
+		(property "Reference" "J9"
 			(at 26.67 87.2955 0)
 			(effects
@@
 			(project "wexlacon"
 				(path "/0fece1c8-c6d0-4b5d-a04d-4f9ff43ff97c"
-					(reference "J4")
+					(reference "J9")
 					(unit 1)
 				)
@@
 		(dnp no)
 		(fields_autoplaced yes)
-		(property "Reference" "J2"
+		(property "Reference" "J1"
 			(at 26.67 19.9855 0)
 			(effects
@@
 			(project ""
 				(path "/0fece1c8-c6d0-4b5d-a04d-4f9ff43ff97c"
-					(reference "J2")
+					(reference "J1")
 					(unit 1)
 				)
@@
 		(dnp no)
 		(fields_autoplaced yes)
-		(property "Reference" "J3"
+		(property "Reference" "J10"
 			(at 26.67 65.7055 0)
 			(effects
@@
 			(project ""
 				(path "/0fece1c8-c6d0-4b5d-a04d-4f9ff43ff97c"
-					(reference "J3")
+					(reference "J10")
 					(unit 1)
 				)

Commit message: Adapter drill d=1.8 mm.
Parts:
- removed H4, H6: 1.0mm, TestPoint:TestPoint_THTPad_D2.0mm_Drill1.0mm, symbol Mechanical:MountingHole
Other:
- note added: "Turnout wire hole"
- note removed: "Turnout wire holes"
Changed lines of the file:
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@@
 		)
 	)
-	(text "Turnout wire\nholes"
+	(text "Turnout wire\nhole"
 		(exclude_from_sim no)
-		(at 69.85 111.76 0)
+		(at 69.85 116.84 0)
 		(effects
 			(font
@@
 	)
 	(symbol
-		(lib_id "Mechanical:MountingHole")
-		(at 66.04 116.84 0)
-		(unit 1)
-		(exclude_from_sim yes)
-		(in_bom no)
-		(on_board yes)
-		(dnp no)
-		(property "Reference" "H4"
-			(at 68.58 116.3708 0)
-			(effects
-				(font
-					(size 1.27 1.27)
-				)
-				(justify left)
-			)
-		)
-		(property "Value" "1.0mm"
-			(at 68.58 118.0522 0)
-			(effects
-				(font
-					(size 1.27 1.27)
-				)
-				(justify left)
-			)
-		)
-		(property "Footprint" "TestPoint:TestPoint_THTPad_D2.0mm_Drill1.0mm"
-			(at 66.04 116.84 0)
-			(effects
-				(font
-					(size 1.27 1.27)
-				)
-				(hide yes)
-			)
-		)
-		(property "Datasheet" "~"
-			(at 66.04 116.84 0)
-			(effects
-				(font
-					(size 1.27 1.27)
-				)
-				(hide yes)
-			)
-		)
-		(property "Description" "Mounting Hole without connection"
-			(at 66.04 116.84 0)
-			(effects
-				(font
-					(size 1.27 1.27)
-				)
-				(hide yes)
-			)
-		)
-		(instances
-			(project ""
-				(path "/0fece1c8-c6d0-4b5d-a04d-4f9ff43ff97c"
-					(reference "H4")
-					(unit 1)
-				)
-			)
-		)
-	)
-	(symbol
 		(lib_id "Connector:DB25_Receptacle")
 		(at 181.61 55.88 0)
@@
 					(unit 1)
 				)
-			)
-		)
-	)
-	(symbol
-		(lib_id "Mechanical:MountingHole")
-		(at 66.04 127 0)
-		(unit 1)
-		(exclude_from_sim yes)
-		(in_bom no)
-		(on_board yes)
-		(dnp no)
-		(fields_autoplaced yes)
-		(property "Reference" "H6"
-			(at 68.58 125.7878 0)
-			(effects
-				(font
-					(size 1.27 1.27)
-				)
-				(justify left)
-			)
-		)
-		(property "Value" "1.0mm"
-			(at 68.58 128.2121 0)
-			(effects
-				(font
-					(size 1.27 1.27)
-				)
-				(justify left)
-			)
-		)
-		(property "Footprint" "TestPoint:TestPoint_THTPad_D2.0mm_Drill1.0mm"
-			(at 66.04 127 0)
-			(effects
-				(font
-					(size 1.27 1.27)
-				)
-				(hide yes)
-			)
-		)
-		(property "Datasheet" "~"
-			(at 66.04 127 0)
-			(effects
-				(font
-					(size 1.27 1.27)
-				)
-				(hide yes)
-			)
-		)
-		(property "Description" "Mounting Hole without connection"
-			(at 66.04 127 0)
-			(effects
-				(font
-					(size 1.27 1.27)
-				)
-				(hide yes)
-			)
-		)
-		(instances
-			(project "wexlacon"
-				(path "/0fece1c8-c6d0-4b5d-a04d-4f9ff43ff97c"
-					(reference "H6")
-					(unit 1)
-				)

Commit message: Fix switched order of relay contacts.
Connections:
- net RELA+: now also J5.24 (P24), J5.25 (P25), J9.3 (Pin_3); no longer J5.20 (P20), J5.21 (P21), J9.1 (Pin_1)
- net RELA-: now also J5.20 (P20), J5.21 (P21), J9.1 (Pin_1); no longer J5.24 (P24), J5.25 (P25), J9.3 (Pin_3)
- net RELB+: now also J10.1 (Pin_1), J5.8, J5.9; no longer J10.3 (Pin_3), J5.12, J5.13
- net RELB-: now also J10.3 (Pin_3), J5.12, J5.13; no longer J10.1 (Pin_1), J5.8, J5.9
